File: STM32L433CBT_Developement_Board/STM32L433CBT_Dev_Board.kicad_pcb (KiCad board)
At the start: 2 copper layers, 26.7 x 48.8 mm, 39 parts, among them J1 USB_B_Micro, J2 Conn_01x18_Male, J3 Conn_01x18_Male, J4 Conn_02x03_Counter_Clockwise, J5 Conn_01x04_Male, J7 USB_B_Micro, SW1 SW_DIP_x01, U1 STM32L433CBTx, U2 CP2102N-A01-GQFN24, U3 W25Q128JVS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

Commit message: Add files via upload
Parts:
- removed C7: C_Small, Capacitor_SMD:C_0805_2012Metric
- removed D1, D2, D3, D4: LED, Diode_SMD:D_0805_2012Metric
- removed D5, D6: NeoPixel_THT, LED_SMD:LED_WS2812B_PLCC4_5.0x5.0mm_P3.2mm
- removed J1: USB_B_Micro, Connector_USB:USB_Micro-B_Molex_47346-0001
- removed J4: Conn_02x03_Counter_Clockwise, Connector_PinHeader_2.54mm:PinHeader_2x03_P2.54mm_Vertical_SMD
- removed J5: Conn_01x04_Male, Connector_PinHeader_2.54mm:PinHeader_1x04_P2.54mm_Horizontal
- removed SW1: SW_DIP_x01, Button_Switch_SMD:SW_SPST_B3U-1000P-B
- removed U1: STM32L433CBTx, Package_QFP:LQFP-48_7x7mm_P0.5mm
- removed U3: W25Q128JVS, Package_SO:SOIC-8_5.23x5.23mm_P1.27mm
- added BOOT: Conn_02x03_Counter_Clockwise, Connector_PinHeader_2.54mm:PinHeader_2x03_P2.54mm_Vertical_SMD, F.Cu at (199.7, 56.4)
- added C14: C_Small, Capacitor_SMD:C_0805_2012Metric, F.Cu at (187.3, 91.1)
- added LED: NeoPixel_THT, LED_SMD:LED_WS2812B_PLCC4_5.0x5.0mm_P3.2mm, F.Cu at (200.7, 87.2)
- added RESET: SW_DIP_x01, Button_Switch_SMD:SW_SPST_B3U-1000P-B, F.Cu at (193.2, 78.9)
- added STM32L433CBT: STM32L433CBTx, Package_QFP:LQFP-48_7x7mm_P0.5mm, F.Cu at (193.8, 68.3)
- added SWD: Conn_01x04_Male, Connector_PinHeader_2.54mm:PinHeader_1x04_P2.54mm_Horizontal, F.Cu at (195.8, 48.8)
- added USB_to_UART: USB_B_Micro, Connector_USB:USB_Micro-B_Molex_47346-0001, F.Cu at (188.2, 47.8)
- added W25Q128: W25Q128JVS, Package_SO:SOIC-8_5.23x5.23mm_P1.27mm, F.Cu at (191.5, 84.6)
- C1, C13, C2, C3, C5, C8, D12, D7, D9, R1, R2, R3, U2: moved to B.Cu
- Y1, Y2: value Crystal -> Crystal_GND23_Small; footprint Crystal:Crystal_SMD_HC49-SD -> Crystal:Crystal_SMD_Abracon_ABM8G-4Pin_3.2x2.5mm
- moved Y1 155.2 mm to (190.3, 58.4), turned to 90 degrees
- moved C6 155.1 mm to (197.1, 81.4), turned to 90 degrees
- moved J2 149.8 mm to (207.0, 49.5)
- moved U4 148.9 mm to (199.4, 56.0), turned to 180 degrees
- moved J7 148.6 mm to (193.8, 92.2)
- moved C4 147.5 mm to (192.8, 52.4), turned to 180 degrees
- moved D9 147.1 mm to (203.2, 88.5)
- moved J3 146.8 mm to (180.8, 49.5)
- moved Y2 146.6 mm to (185.5, 58.3), turned to 90 degrees
- moved C5 143.8 mm to (201.3, 51.5), turned to 180 degrees
- moved R2 139.3 mm to (193.2, 60.1), turned to 270 degrees
- moved D7 136.8 mm to (200.6, 91.3)
- moved C9 133.9 mm to (183.8, 54.1), turned to 90 degrees
- moved C12 133.8 mm to (193.1, 56.0), turned to 90 degrees
- moved C10 133.6 mm to (185.9, 54.1), turned to 90 degrees
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Connections:
- C10 pad 1: /OSC8_OUT -> /OSC8_IN
- C11 pad 1: /OSC32_IN -> /OSC32_OUT
- C12 pad 1: /OSC32_OUT -> /OSC32_IN
- C9 pad 1: /OSC8_IN -> /OSC8_OUT
- D7 pad 1: /D+ -> /D-
- J2 pad 14: /PB0 -> GND
- U2 pad 3: Net-(D1-Pad2) -> /D+
- U2 pad 4: Net-(D2-Pad2) -> /D-
- Y1 pad 1: /OSC8_IN -> /OSC32_IN
- Y1 pad 2: /OSC8_OUT -> GND
- Y2 pad 1: /OSC32_IN -> /OSC8_IN
- Y2 pad 2: /OSC32_OUT -> GND
Routing:
- net +5V: track 41.5 -> 192.8 mm, vias 0 -> 5
- net +3V3: track 48.5 -> 88.9 mm, vias 2 -> 3
- net /PA9: track 0.00 -> 36.1 mm, vias 0 -> 1
- net /PA10: track 0.00 -> 33.7 mm, vias 0 -> 1
- net /D-: track 9.95 -> 39.6 mm, vias 0 -> 3
- net /D+: track 10.7 -> 36.4 mm, vias 0 -> 3
- net /PC13: track 25.5 -> 49.7 mm
- net /PA13: track 42.3 -> 23.1 mm, vias 1 -> 2
- net /PA14: track 37.0 -> 19.7 mm, vias 1 -> 0
- net /PB0: track 32.3 -> 15.6 mm, vias 2 -> 0
- net /PA8: track 0.00 -> 16.1 mm
- net /PA7: track 16.6 -> 30.7 mm, vias 0 -> 1
- net /PB11: track 11.7 -> 24.7 mm
- net /PA5: track 16.3 -> 29.3 mm, vias 0 -> 2
- net /PB12: track 13.3 -> 24.9 mm, vias 2 -> 0
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- added copper zone on B.Cu, net GND
- added copper zone on F.Cu, net GND
Other:
- board size 26.7 x 48.8 mm -> 30.2 x 50.3 mm
- board text added: "+3.3V"
- board text added: "+5V"
- board text added: "32 KHz"
- board text added: "8 MHz"
- board text added: "BOOT0"
- board text added: "BOOT1"
- board text added: "GND"
- board text added: "PA0"
- board text added: "PA1"
- board text added: "PA10"
- board text added: "PA15"
- board text added: "PA2"
- board text added: "PA3"
- board text added: "PA4"
- board text added: "PA5"
- board text added: "PA6"
- board text added: "PA7"
- board text added: "PA8"
- board text added: "PA9"
- board text added: "PB0"
- board text added: "PB1"
- board text added: "PB10"
- board text added: "PB11"
- board text added: "PB12"
- board text added: "PB13"
- board text added: "PB14"
- board text added: "PB15"
- board text added: "PB2"
- board text added: "PB3"
- board text added: "PB4"
- board text added: "PB5"
- board text added: "PB6"
- board text added: "PB7"
- board text added: "PB8"
- board text added: "PB9"
- board text added: "PC13"
- board text added: "SWCLK"
- board text added: "SWDIO"
- board text added: "USB"

Commit message: Add files via upload
Parts:
- moved C5 70.5 mm to (139.5, 85.5)
- moved C1 70.5 mm to (133.4, 95.2)
- moved C10 70.5 mm to (124.1, 88.0)
- moved C11 70.5 mm to (126.2, 88.8)
- moved C13 70.5 mm to (133.4, 109.2)
- moved C14 70.5 mm to (125.5, 125.0)
- moved C2 70.5 mm to (123.8, 88.3)
- moved C3 70.5 mm to (124.5, 85.8)
- moved D10 70.5 mm to (142.8, 85.3)
- moved D7 70.5 mm to (138.8, 125.2)
- moved J3 70.5 mm to (119.0, 83.4)
- moved LED 70.5 mm to (138.8, 121.0)
- moved R1 70.5 mm to (132.1, 90.3)
- moved R2 70.5 mm to (131.3, 94.0)
- moved R3 70.5 mm to (135.7, 111.3)
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Routing:
- net GND: track 9.89 -> 280.7 mm, vias 0 -> 4
- net +5V: track 192.8 -> 125.5 mm, vias 5 -> 3
- net /D-: track 39.6 -> 101.9 mm
- net +3V3: track 88.9 -> 130.6 mm, vias 3 -> 4
- net /D+: track 36.4 -> 67.8 mm, vias 3 -> 5
- net /PA13: track 23.1 -> 42.0 mm, vias 2 -> 0
- net /PA10: track 33.7 -> 49.4 mm, vias 1 -> 0
- net /PA14: track 19.7 -> 34.2 mm
- net /PA4: track 24.3 -> 33.5 mm, vias 1 -> 0
- net /PA15: track 12.1 -> 20.6 mm, vias 2 -> 1
- net /PA9: track 36.1 -> 44.3 mm, vias 1 -> 0
- net /NRST: track 26.0 -> 18.8 mm, vias 3 -> 2
- net /PA1: track 9.53 -> 15.6 mm
- net /PC13: track 49.7 -> 44.2 mm
- net /BOOT0: track 2.15 -> 6.79 mm, vias 1 -> 2
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