File: Project X/Project X.kicad_pcb (KiCad board)
At the start: 2 copper layers, 30 x 70.1 mm, 45 parts, among them IC1 W25Q128JVPIQ, J1 Conn_01x04, J2 Conn_01x26, J3 Conn_01x26, P1 USB_C_Plug_USB2.0, SW1 SW_SPST, SW2 SW_SPST, SW3 SW_SPST, U1 LT1129-3.3_SOT223, U2 STM32L476RCTx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

Commit message: Add files via upload
Parts:
- C10, IC1: moved to B.Cu
- moved C15 105.2 mm to (102.8, 133.3)
- moved C17 105.2 mm to (98.1, 135.8)
- moved C19 105.2 mm to (99.1, 135.9)
- moved U3 105.2 mm to (98.9, 132.0)
- moved C20 103.8 mm to (106.9, 90.6)
- moved R6 103.8 mm to (106.9, 92.9)
- moved SW2 103.8 mm to (109.4, 88.4)
- moved C18 103.4 mm to (110.5, 130.2), turned to 180 degrees
- moved SW3 102.0 mm to (97.0, 88.4)
- moved C21 102.0 mm to (94.8, 90.5)
- moved R7 102.0 mm to (94.8, 92.5)
- moved SW1 97.9 mm to (112.7, 132.6), turned to 270 degrees
- moved R4 94.2 mm to (101.9, 97.6)
- moved D1 94.2 mm to (99.7, 97.6)
- moved R3 91.7 mm to (115.3, 135.5), turned to 90 degrees
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Routing:
- net GND: track 0.00 -> 323.8 mm, vias 0 -> 2
- net +3V3: track 0.00 -> 185.0 mm, vias 0 -> 7
- net +5V: track 0.00 -> 59.9 mm
- net /PB13: track 0.00 -> 55.2 mm
- net /PA1: track 0.00 -> 50.2 mm
- net /PA2: track 0.00 -> 50.1 mm, vias 0 -> 1
- net /PA4: track 0.00 -> 49.5 mm, vias 0 -> 1
- net /D+: track 0.00 -> 41.7 mm, vias 0 -> 1
- net /SWDIO: track 0.00 -> 41.7 mm
- net /D-: track 0.00 -> 40.6 mm, vias 0 -> 1
- net /NRST: track 0.02 -> 40.3 mm, vias 0 -> 1
- net /PB14: track 0.00 -> 39.2 mm
- net /PA5: track 0.00 -> 37.6 mm, vias 0 -> 2
- net /PB12: track 0.00 -> 37.5 mm, vias 0 -> 1
- net /PC0: track 0.00 -> 37.2 mm, vias 0 -> 1
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- added copper zone on B.Cu, net GND
- added copper zone on F.Cu, net GND
Other:
- board size 30 x 70.1 mm -> 30 x 74.4 mm
- board text added: "+3.3v"
- board text added: "+5V"
- board text added: "GND"

Commit message: Add files via upload
Parts:
- added REF**: MountingHole_2.2mm_M2_DIN965_Pad, MountingHole:MountingHole_2.2mm_M2_DIN965_Pad, F.Cu at (96.5, 85.5)
- added REF**: MountingHole_2.2mm_M2_DIN965_Pad, MountingHole:MountingHole_2.2mm_M2_DIN965_Pad, F.Cu at (96.5, 110.0)
- added mouse-bite-2mm-slot: VAL**, ASSETS:mouse-bite-2mm-slot, F.Cu at (252.8, 119.8)
- moved P1 80.3 mm to (164.8, 97.8), turned to 90 degrees
- moved C16 68.7 mm to (156.2, 99.2), turned to 0 degrees
- moved R1 66.5 mm to (154.6, 100.5), turned to 270 degrees
- moved R2 66.2 mm to (154.6, 98.0), turned to 270 degrees
- moved C10 63.4 mm to (152.3, 100.5), turned to 90 degrees
- moved IC1 61.7 mm to (150.4, 104.8), turned to 90 degrees
- moved C17 57.9 mm to (147.6, 105.7), turned to 0 degrees
- moved C19 57.7 mm to (147.7, 104.7), turned to 180 degrees
- moved R3 56.9 mm to (147.2, 88.5), turned to 180 degrees
- moved C15 53.2 mm to (145.1, 100.9), turned to 90 degrees
- moved U3 52.4 mm to (143.8, 104.8), turned to 90 degrees
- moved SW1 52.2 mm to (144.3, 91.0), turned to 0 degrees
- moved C18 48.5 mm to (141.9, 93.2), turned to 270 degrees
- moved C4 39.3 mm to (135.0, 101.4), turned to 135 degrees
- moved C8 35.0 mm to (130.4, 106.0), turned to 315 degrees
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- renumbered SW3 to Button1, SW2 to Button2
Routing:
- net +3V3: track 185.0 -> 187.2 mm
- net Net-(P1-PadA4): track 12.8 -> 14.5 mm
- net /PB13: track 55.2 -> 56.0 mm
Other:
- board size 30 x 74.4 mm -> 74.4 x 30 mm
- board text added: "+3.3V"
- board text added: "By Kunal Salvi"
- board text added: "PA0"
- board text added: "PA1"
- board text added: "PA10"
- board text added: "PA15"
- board text added: "PA2"
- board text added: "PA3"
- board text added: "PA4"
- board text added: "PA5"
- board text added: "PA6"
- board text added: "PA7"
- board text added: "PA8"
- board text added: "PA9"
- board text added: "PB0"
- board text added: "PB1"
- board text added: "PB10"
- board text added: "PB11"
- board text added: "PB12"
- board text added: "PB13"
- board text added: "PB14"
- board text added: "PB15"
- board text added: "PB2"
- board text added: "PB3"
- board text added: "PB4"
- board text added: "PB5"
- board text added: "PB6"
- board text added: "PB7"
- board text added: "PB8"
- board text added: "PB9"
- board text added: "PC0"
- board text added: "PC1"
- board text added: "PC10"
- board text added: "PC11"
- board text added: "PC12"
- board text added: "PC13"
- board text added: "PC2"
- board text added: "PC3"
- board text added: "PC4"
- board text added: "PC5"
- board text added: "PC6"
- board text added: "PC7"
- board text added: "PC8"
- board text added: "PC9"
- board text added: "PD2"
- board text added: "Reset"
- board text added: "SWCLK"
- board text added: "SWDIO"
