File: STM32G473RET6 Development Board/MPU9250.sch (KiCad schematic (older format))
At the start: 0 parts

Commit message: Add files via upload
Parts:
- added C? (x3): C_Small, symbol Device:C_Small
- added D?: LED, symbol Device:LED
- added R?: R_Small, symbol Device:R_Small
- added U?: MPU-9250, Sensor_Motion:InvenSense_QFN-24_3x3mm_P0.4mm, symbol Sensor_Motion:MPU-9250
Connections:
- new net: C?.2, U?.10 (REGOUT)
- new net: D?.2 (A), R?.2
- new net +3.3V: C?.2, C?.2, R?.1, U?.13 (VDD), U?.8 (VDDIO)
- new net +3.3v: U?.1 (RESV_VDDIO)
- new net GND: C?.1, C?.1, C?.1, U?.18 (GND), U?.20 (RESV_GND)
- new net PA2: U?.12 (INT)
- new net PA3: U?.11 (FSYNC)
- new net PA4: D?.1 (K), U?.22 (~CS)
- new net PA5: U?.23 (SCL/SCLK)
- new net PA6: U?.9 (AD0/MISO)
- new net PA7: U?.24 (SDA/MOSI)
- no-connect marks 0 -> 2
Changed lines of the file:
@@
 Sheet 7 7
 Title ""
-Date ""
-Rev ""
+Date "2020-04-03"
+Rev "1"
 Comp ""
 Comment1 ""
@@
 Comment4 ""
 $EndDescr
+$Comp
+L Sensor_Motion:MPU-9250 U?
+U 1 1 5EC32462
+P 4050 3600
+F 0 "U?" H 4600 4450 50  0000 C CNN
+F 1 "MPU-9250" H 4600 4350 50  0000 C CNN
+F 2 "Sensor_Motion:InvenSense_QFN-24_3x3mm_P0.4mm" H 4050 2600 50  0001 C CNN
+F 3 "https://store.invensense.com/datasheets/invensense/MPU9250REV1.0.pdf" H 4050 3450 50  0001 C CNN
+	1    4050 3600
+	1    0    0    -1
+$EndComp
+Text GLabel 2700 3600 0    50   Input ~ 0
+PA4
+Text GLabel 3200 3400 0    50   Input ~ 0
+PA6
+Text GLabel 3200 3300 0    50   Input ~ 0
+PA7
+Text GLabel 3200 3500 0    50   Input ~ 0
+PA5
+Text GLabel 3650 2350 0    50   Input ~ 0
++3.3V
+Text GLabel 3200 3800 0    50   Input ~ 0
+PA3
+Text GLabel 4900 3300 2    50   Input ~ 0
+PA2
+Wire Wire Line
+	4900 3300 4750 3300
+Wire Wire Line
+	3350 3300 3200 3300
+Wire Wire Line
+	3200 3400 3350 3400
+Wire Wire Line
+	3350 3500 3200 3500
+Wire Wire Line
+	3200 3800 3350 3800
+Wire Wire Line
+	4050 4500 4050 4700
+$Comp
+L power:GND #PWR?
+U 1 1 5EC41280
+P 4050 4700
+F 0 "#PWR?" H 4050 4450 50  0001 C CNN
+F 1 "GND" H 4055 4527 50  0000 C CNN
+F 2 "" H 4050 4700 50  0001 C CNN
+F 3 "" H 4050 4700 50  0001 C CNN
+	1    4050 4700
+	1    0    0    -1
+$EndComp
+Wire Wire Line
+	3950 2700 3950 2550
+Wire Wire Line
+	3950 2350 3650 2350
+Text GLabel 4350 2350 2    50   Input ~ 0
++3.3V
+Wire Wire Line
+	4350 2350 4150 2350
+Wire Wire Line
+	4150 2350 4150 2550
+NoConn ~ 4750 3500
+NoConn ~ 4750 3600
+$Comp
+L Device:C_Small C?
+U 1 1 5E8738DF
+P 5000 2550
+F 0 "C?" V 4771 2550 50  0000 C CNN
+F 1 "C_Small" V 4862 2550 50  0000 C CNN
+F 2 "" H 5000 2550 50  0001 C CNN
+F 3 "~" H 5000 2550 50  0001 C CNN
+	1    5000 2550
+	0    1    1    0
+$EndComp
+Wire Wire Line
+	4900 2550 4150 2550
+Connection ~ 4150 2550
+Wire Wire Line
+	4150 2550 4150 2700
+Wire Wire Line
+	5100 2550 5450 2550
+Wire Wire Line
+	5450 2550 5450 2700
+$Comp
+L power:GND #PWR?
+U 1 1 5E87481B
+P 5450 2700
+F 0 "#PWR?" H 5450 2450 50  0001 C CNN
+F 1 "GND" H 5455 2527 50  0000 C CNN
+F 2 "" H 5450 2700 50  0001 C CNN
+F 3 "" H 5450 2700 50  0001 C CNN
+	1    5450 2700
+	1    0    0    -1
+$EndComp
+$Comp
+L Device:C_Small C?
+U 1 1 5E875BB1
+P 3050 2550
+F 0 "C?" V 2821 2550 50  0000 C CNN
+F 1 "C_Small" V 2912 2550 50  0000 C CNN
+F 2 "" H 3050 2550 50  0001 C CNN
+F 3 "~" H 3050 2550 50  0001 C CNN
+	1    3050 2550
+	0    -1   1    0
+$EndComp
+Wire Wire Line
+	2950 2550 2600 2550
+Wire Wire Line
+	2600 2550 2600 2700
+$Comp
+L power:GND #PWR?
+U 1 1 5E875BBA
+P 2600 2700
+F 0 "#PWR?" H 2600 2450 50  0001 C CNN
+F 1 "GND" H 2605 2527 50  0000 C CNN
+F 2 "" H 2600 2700 50  0001 C CNN
+F 3 "" H 2600 2700 50  0001 C CNN
+	1    2600 2700
+	-1   0    0    -1
+$EndComp
+Wire Wire Line
+	3150 2550 3950 2550
+Connection ~ 3950 2550
+Wire Wire Line
+	3950 2550 3950 2350
+$Comp
+L Device:C_Small C?
+U 1 1 5E876306
+P 5400 3800
+F 0 "C?" V 5171 3800 50  0000 C CNN
+F 1 "C_Small" V 5262 3800 50  0000 C CNN
+F 2 "" H 5400 3800 50  0001 C CNN
+F 3 "~" H 5400 3800 50  0001 C CNN
+	1    5400 3800
+	0    1    1    0
+$EndComp
+Wire Wire Line
+	5300 3800 4750 3800
+Wire Wire Line
+	5500 3800 5850 3800
+Wire Wire Line
+	5850 3800 5850 3900
+$Comp
+L power:GND #PWR?
+U 1 1 5E877A1A
+P 5850 3900
+F 0 "#PWR?" H 5850 3650 50  0001 C CNN
+F 1 "GND" H 5855 3727 50  0000 C CNN
+F 2 "" H 5850 3900 50  0001 C CNN
+F 3 "" H 5850 3900 50  0001 C CNN
+	1    5850 3900
+	1    0    0    -1
+$EndComp
+Text GLabel 5000 3900 2    50   Input ~ 0
++3.3v
+Wire Wire Line
+	5000 3900 4750 3900
+Wire Wire Line
+	4750 4000 4950 4000
+Wire Wire Line
+	4950 4000 4950 4100
+$Comp
+L power:GND #PWR?
+U 1 1 5E878A2B
+P 4950 4100
+F 0 "#PWR?" H 4950 3850 50  0001 C CNN
+F 1 "GND" H 4955 3927 50  0000 C CNN
+F 2 "" H 4950 4100 50  0001 C CNN
+F 3 "" H 4950 4100 50  0001 C CNN
+	1    4950 4100
+	1    0    0    -1
+$EndComp
+Wire Wire Line
+	2700 3600 2800 3600
+$Comp
+L Device:LED D?
+U 1 1 5E8A70FB
+P 2800 3250
+F 0 "D?" V 2850 3450 50  0000 R CNN
+F 1 "LED" V 2750 3450 50  0000 R CNN
+F 2 "" H 2800 3250 50  0001 C CNN
+F 3 "~" H 2800 3250 50  0001 C CNN
+	1    2800 3250
+	0    -1   -1   0
+$EndComp
+$Comp
+L Device:R_Small R?
+U 1 1 5E8A85A6
+P 2800 2900
+F 0 "R?" H 2859 2946 50  0000 L CNN
+F 1 "R_Small" H 2859 2855 50  0000 L CNN
+F 2 "" H 2800 2900 50  0001 C CNN
+F 3 "~" H 2800 2900 50  0001 C CNN
+	1    2800 2900
+	1    0    0    -1
+$EndComp
+Wire Wire Line
+	2800 3000 2800 3100
+Wire Wire Line
+	2800 3400 2800 3600
+Connection ~ 2800 3600
+Wire Wire Line
+	2800 3600 3350 3600
+Wire Wire Line
+	2800 2800 2800 2750
+Wire Wire Line
+	2800 2750 2950 2750
+Text GLabel 2950 2750 2    50   Input ~ 0
++3.3V
 $EndSCHEMATC

Commit message: Add files via upload
Parts:
- C26, C27, C28: renamed from C?; footprint (none) -> Capacitor_SMD:C_0402_1005Metric
- D5: renamed from D?; footprint (none) -> LED_SMD:LED_0805_2012Metric_Pad1.15x1.40mm_HandSolder
- R18: renamed from R?; footprint (none) -> Resistor_SMD:R_0603_1608Metric
- gave numbers to parts that had none: 1
Connections:
- net +3.3v is gone; now on net +3.3V: U4.1 (RESV_VDDIO)
Changed lines of the file:
@@
 $EndDescr
 $Comp
-L Sensor_Motion:MPU-9250 U?
+L Sensor_Motion:MPU-9250 U4
 U 1 1 5EC32462
 P 4050 3600
-F 0 "U?" H 4600 4450 50  0000 C CNN
+F 0 "U4" H 4600 4450 50  0000 C CNN
 F 1 "MPU-9250" H 4600 4350 50  0000 C CNN
 F 2 "Sensor_Motion:InvenSense_QFN-24_3x3mm_P0.4mm" H 4050 2600 50  0001 C CNN
@@
 	4050 4500 4050 4700
 $Comp
-L power:GND #PWR?
+L power:GND #PWR0147
 U 1 1 5EC41280
 P 4050 4700
-F 0 "#PWR?" H 4050 4450 50  0001 C CNN
+F 0 "#PWR0147" H 4050 4450 50  0001 C CNN
 F 1 "GND" H 4055 4527 50  0000 C CNN
 F 2 "" H 4050 4700 50  0001 C CNN
@@
 NoConn ~ 4750 3600
 $Comp
-L Device:C_Small C?
+L Device:C_Small C27
 U 1 1 5E8738DF
 P 5000 2550
-F 0 "C?" V 4771 2550 50  0000 C CNN
+F 0 "C27" V 4771 2550 50  0000 C CNN
 F 1 "C_Small" V 4862 2550 50  0000 C CNN
-F 2 "" H 5000 2550 50  0001 C CNN
+F 2 "Capacitor_SMD:C_0402_1005Metric" H 5000 2550 50  0001 C CNN
 F 3 "~" H 5000 2550 50  0001 C CNN
 	1    5000 2550
@@
 	5450 2550 5450 2700
 $Comp
-L power:GND #PWR?
+L power:GND #PWR0148
 U 1 1 5E87481B
 P 5450 2700
-F 0 "#PWR?" H 5450 2450 50  0001 C CNN
+F 0 "#PWR0148" H 5450 2450 50  0001 C CNN
 F 1 "GND" H 5455 2527 50  0000 C CNN
 F 2 "" H 5450 2700 50  0001 C CNN
@@
 $EndComp
 $Comp
-L Device:C_Small C?
+L Device:C_Small C26
 U 1 1 5E875BB1
 P 3050 2550
-F 0 "C?" V 2821 2550 50  0000 C CNN
+F 0 "C26" V 2821 2550 50  0000 C CNN
 F 1 "C_Small" V 2912 2550 50  0000 C CNN
-F 2 "" H 3050 2550 50  0001 C CNN
+F 2 "Capacitor_SMD:C_0402_1005Metric" H 3050 2550 50  0001 C CNN
 F 3 "~" H 3050 2550 50  0001 C CNN
 	1    3050 2550
@@
 	2600 2550 2600 2700
 $Comp
-L power:GND #PWR?
+L power:GND #PWR0149
 U 1 1 5E875BBA
 P 2600 2700
-F 0 "#PWR?" H 2600 2450 50  0001 C CNN
+F 0 "#PWR0149" H 2600 2450 50  0001 C CNN
 F 1 "GND" H 2605 2527 50  0000 C CNN
 F 2 "" H 2600 2700 50  0001 C CNN
@@
 	3950 2550 3950 2350
 $Comp
-L Device:C_Small C?
+L Device:C_Small C28
 U 1 1 5E876306
 P 5400 3800
-F 0 "C?" V 5171 3800 50  0000 C CNN
+F 0 "C28" V 5171 3800 50  0000 C CNN
 F 1 "C_Small" V 5262 3800 50  0000 C CNN
-F 2 "" H 5400 3800 50  0001 C CNN
+F 2 "Capacitor_SMD:C_0402_1005Metric" H 5400 3800 50  0001 C CNN
 F 3 "~" H 5400 3800 50  0001 C CNN
 	1    5400 3800
@@
 	5850 3800 5850 3900
 $Comp
-L power:GND #PWR?
+L power:GND #PWR0150
 U 1 1 5E877A1A
 P 5850 3900
-F 0 "#PWR?" H 5850 3650 50  0001 C CNN
+F 0 "#PWR0150" H 5850 3650 50  0001 C CNN
 F 1 "GND" H 5855 3727 50  0000 C CNN
 F 2 "" H 5850 3900 50  0001 C CNN
@@
 $EndComp
 Text GLabel 5000 3900 2    50   Input ~ 0
-+3.3v
++3.3V
 Wire Wire Line
 	5000 3900 4750 3900
@@
 	4950 4000 4950 4100
 $Comp
-L power:GND #PWR?
+L power:GND #PWR0151
 U 1 1 5E878A2B
 P 4950 4100
-F 0 "#PWR?" H 4950 3850 50  0001 C CNN
+F 0 "#PWR0151" H 4950 3850 50  0001 C CNN
 F 1 "GND" H 4955 3927 50  0000 C CNN
 F 2 "" H 4950 4100 50  0001 C CNN
@@
 	2700 3600 2800 3600
 $Comp
-L Device:LED D?
+L Device:LED D5
 U 1 1 5E8A70FB
 P 2800 3250
-F 0 "D?" V 2850 3450 50  0000 R CNN
+F 0 "D5" V 2850 3450 50  0000 R CNN
 F 1 "LED" V 2750 3450 50  0000 R CNN
-F 2 "" H 2800 3250 50  0001 C CNN
+F 2 "LED_SMD:LED_0805_2012Metric_Pad1.15x1.40mm_HandSolder" H 2800 3250 50  0001 C CNN
 F 3 "~" H 2800 3250 50  0001 C CNN
 	1    2800 3250
@@
 $EndComp
 $Comp
-L Device:R_Small R?
+L Device:R_Small R18
 U 1 1 5E8A85A6
 P 2800 2900
-F 0 "R?" H 2859 2946 50  0000 L CNN
+F 0 "R18" H 2859 2946 50  0000 L CNN
 F 1 "R_Small" H 2859 2855 50  0000 L CNN
-F 2 "" H 2800 2900 50  0001 C CNN
+F 2 "Resistor_SMD:R_0603_1608Metric" H 2800 2900 50  0001 C CNN
 F 3 "~" H 2800 2900 50  0001 C CNN
 	1    2800 2900
