File: STM32G473RET6 Development Board/Connectors.sch (KiCad schematic (older format))
At the start: 0 parts

Commit message: Add files via upload
Parts:
- added C? (x2): C_Small, symbol Device:C_Small
- added J? (x2): Conn_01x04, symbol Connector_Generic:Conn_01x04
- added J? (x2): Conn_01x23, symbol Connector_Generic:Conn_01x23
- added J?: Conn_02x02_Top_Bottom, symbol Connector_Generic:Conn_02x02_Top_Bottom
- added R? (x2): 4.7k, symbol Device:R_Small
Connections:
- new net +3.3V: C?.2, C?.2, J?.1 (Pin_1), J?.1 (Pin_1), J?.1 (Pin_1)
- new net +5V: J?.3 (Pin_3)
- new net 3+3.3V: R?.1, R?.1
- new net GND: C?.1, C?.1, J?.2 (Pin_2), J?.4 (Pin_4), J?.4 (Pin_4), J?.4 (Pin_4)
- new net PA0: J?.6 (Pin_6)
- new net PA1: J?.7 (Pin_7)
- new net PA10: J?.17 (Pin_17)
- new net PA11: J?.16 (Pin_16)
- new net PA12: J?.15 (Pin_15)
- new net PA13: J?.1 (Pin_1), J?.2 (Pin_2)
- new net PA14: J?.2 (Pin_2), J?.3 (Pin_3)
- new net PA15: J?.3 (Pin_3)
- new net PA2: J?.8 (Pin_8)
- new net PA3: J?.9 (Pin_9)
- new net PA4: J?.10 (Pin_10)
- new net PA5: J?.11 (Pin_11)
- new net PA6: J?.12 (Pin_12)
- new net PA7: J?.13 (Pin_13)
- new net PA8: J?.19 (Pin_19)
- new net PA9: J?.18 (Pin_18)
- new net PB0: J?.16 (Pin_16)
- new net PB1: J?.17 (Pin_17)
- new net PB11: J?.19 (Pin_19)
- new net PB12: J?.20 (Pin_20)
- new net PB13: J?.21 (Pin_21)
- new net PB14: J?.22 (Pin_22)
- new net PB15: J?.23 (Pin_23)
- new net PB2: J?.18 (Pin_18)
- new net PB3: J?.8 (Pin_8)
- new net PB4: J?.9 (Pin_9)
- new net PB5: J?.10 (Pin_10)
- new net PB6: J?.11 (Pin_11)
- new net PB7: J?.12 (Pin_12), J?.2 (Pin_2), R?.2
- new net PB8: J?.13 (Pin_13), J?.3 (Pin_3), R?.2
- new net PB9: J?.14 (Pin_14)
- new net PC0: J?.2 (Pin_2)
- new net PC1: J?.3 (Pin_3)
- new net PC10: J?.4 (Pin_4)
- new net PC11: J?.5 (Pin_5)
- new net PC12: J?.6 (Pin_6)
- new net PC13: J?.1 (Pin_1)
- new net PC2: J?.4 (Pin_4)
- new net PC3: J?.5 (Pin_5)
- new net PC4: J?.14 (Pin_14)
- new net PC5: J?.15 (Pin_15)
- new net PC6: J?.23 (Pin_23)
- new net PC7: J?.22 (Pin_22)
- new net PC8: J?.21 (Pin_21)
- new net PC9: J?.20 (Pin_20)
- new net PD2: J?.7 (Pin_7)
Other:
- note added: "SCL\n"
- note added: "SDA"
- note added: "SWCLK"
- note added: "SWDIO\n"

Commit message: Add files via upload
Parts:
- added J8: Conn_ARM_JTAG_SWD_10, Connector_PinHeader_1.27mm:PinHeader_2x05_P1.27mm_Vertical_SMD, symbol Connector:Conn_ARM_JTAG_SWD_10
- C24, C25: renamed from C?; footprint (none) -> Capacitor_SMD:C_0402_1005Metric
- J3, J6: renamed from J?; footprint (none) -> Connector_PinHeader_2.54mm:PinHeader_1x23_P2.54mm_Vertical
- J4, J5: renamed from J?; footprint (none) -> Connector_JST:JST_PH_S4B-PH-K_1x04_P2.00mm_Horizontal
- J7: renamed from J?; footprint (none) -> Connector_PinHeader_2.54mm:PinHeader_2x02_P2.54mm_Vertical
- R16, R17: renamed from R?; footprint (none) -> Resistor_SMD:R_0603_1608Metric
Connections:
- net 3+3.3V is gone; now on net +3.3V: R16.1, R17.1
- net +5V: now also J8.1 (VTref)
- net GND: now also J8.3 (GND), J8.5 (GND), J8.9 (GNDDetect)
- net PA13: now also J8.2 (SWDIO/TMS)
- net PA14: now also J8.4 (SWDCLK/TCK)
- net PB3: now also J8.6 (SWO/TDO)
- new net NRST: J8.10 (~RESET~)
- no-connect marks 0 -> 1
Other:
- note added: "SWCLK\n"
- note added: "SWDIO"
- moved on the sheet: J3

Commit message: Add files via upload
Parts:
- removed R16, R17: 4.7k, Resistor_SMD:R_0603_1608Metric, symbol Device:R_Small
- added R? (x2): 4.7K, Resistor_SMD:R_0603_1608Metric, symbol Device:R_Small
Connections:
- net +3.3V: now also R?.1, R?.1
- net PB7: now also R?.2
- net PB8: now also R?.2
Other:
- moved on the sheet: C25, J5
Changed lines of the file:
@@
 L Connector_Generic:Conn_01x04 J5
 U 1 1 5E88556A
-P 4500 1350
-F 0 "J5" H 4580 1342 50  0000 L CNN
-F 1 "Conn_01x04" H 4580 1251 50  0000 L CNN
-F 2 "Connector_JST:JST_PH_S4B-PH-K_1x04_P2.00mm_Horizontal" H 4500 1350 50  0001 C CNN
-F 3 "~" H 4500 1350 50  0001 C CNN
-	1    4500 1350
-	1    0    0    -1
-$EndComp
-Wire Wire Line
-	4300 1250 4100 1250
-Text GLabel 3900 1250 0    50   Input ~ 0
+P 4500 1400
+F 0 "J5" H 4580 1392 50  0000 L CNN
+F 1 "Conn_01x04" H 4580 1301 50  0000 L CNN
+F 2 "Connector_JST:JST_PH_S4B-PH-K_1x04_P2.00mm_Horizontal" H 4500 1400 50  0001 C CNN
+F 3 "~" H 4500 1400 50  0001 C CNN
+	1    4500 1400
+	1    0    0    -1
+$EndComp
+Wire Wire Line
+	4300 1300 4100 1300
+Text GLabel 3900 1300 0    50   Input ~ 0
 +3.3V
-Text GLabel 3350 1350 0    50   Input ~ 0
+Text GLabel 3350 1400 0    50   Input ~ 0
 PB7
-Text GLabel 3350 1450 0    50   Input ~ 0
+Text GLabel 3350 1500 0    50   Input ~ 0
 PB8
 Wire Wire Line
-	4300 1550 3900 1550
-Wire Wire Line
-	3900 1550 3900 1600
+	4300 1600 3900 1600
+Wire Wire Line
+	3900 1600 3900 1650
 $Comp
 L power:GND #PWR0143
 U 1 1 5E885578
-P 3900 1600
-F 0 "#PWR0143" H 3900 1350 50  0001 C CNN
-F 1 "GND" H 3905 1427 50  0000 C CNN
-F 2 "" H 3900 1600 50  0001 C CNN
-F 3 "" H 3900 1600 50  0001 C CNN
-	1    3900 1600
+P 3900 1650
+F 0 "#PWR0143" H 3900 1400 50  0001 C CNN
+F 1 "GND" H 3905 1477 50  0000 C CNN
+F 2 "" H 3900 1650 50  0001 C CNN
+F 3 "" H 3900 1650 50  0001 C CNN
+	1    3900 1650
 	1    0    0    -1
 $EndComp
@@
 L Device:C_Small C25
 U 1 1 5E88557E
-P 4300 900
-F 0 "C25" V 4071 900 50  0000 C CNN
-F 1 "C_Small" V 4162 900 50  0000 C CNN
-F 2 "Capacitor_SMD:C_0402_1005Metric" H 4300 900 50  0001 C CNN
-F 3 "~" H 4300 900 50  0001 C CNN
-	1    4300 900
+P 4300 950
+F 0 "C25" V 4071 950 50  0000 C CNN
+F 1 "C_Small" V 4162 950 50  0000 C CNN
+F 2 "Capacitor_SMD:C_0402_1005Metric" H 4300 950 50  0001 C CNN
+F 3 "~" H 4300 950 50  0001 C CNN
+	1    4300 950
 	0    1    1    0
 $EndComp
 Wire Wire Line
-	4200 900  4100 900
-Wire Wire Line
-	4100 900  4100 1250
-Connection ~ 4100 1250
-Wire Wire Line
-	4100 1250 3900 1250
-Wire Wire Line
-	4400 900  4750 900
-Wire Wire Line
-	4750 900  4750 1000
+	4200 950  4100 950
+Wire Wire Line
+	4100 950  4100 1300
+Connection ~ 4100 1300
+Wire Wire Line
+	4100 1300 3900 1300
+Wire Wire Line
+	4400 950  4750 950
+Wire Wire Line
+	4750 950  4750 1050
 $Comp
 L power:GND #PWR0144
 U 1 1 5E88558A
-P 4750 1000
-F 0 "#PWR0144" H 4750 750 50  0001 C CNN
-F 1 "GND" H 4755 827 50  0000 C CNN
-F 2 "" H 4750 1000 50  0001 C CNN
-F 3 "" H 4750 1000 50  0001 C CNN
-	1    4750 1000
-	1    0    0    -1
-$EndComp
-Text Notes 3000 1400 0    50   ~ 0
+P 4750 1050
+F 0 "#PWR0144" H 4750 800 50  0001 C CNN
+F 1 "GND" H 4755 877 50  0000 C CNN
+F 2 "" H 4750 1050 50  0001 C CNN
+F 3 "" H 4750 1050 50  0001 C CNN
+	1    4750 1050
+	1    0    0    -1
+$EndComp
+Text Notes 3000 1450 0    50   ~ 0
 SDA
-Text Notes 3000 1500 0    50   ~ 0
+Text Notes 3000 1550 0    50   ~ 0
 SCL\n
 Text Notes 850  1400 0    50   ~ 0
@@
 	500  2000 7350 2000
 Wire Wire Line
-	3350 1350 3450 1350
-Wire Wire Line
-	3350 1450 3500 1450
-$Comp
-L Device:R_Small R17
-U 1 1 5E89E790
-P 3400 850
-F 0 "R17" H 3500 900 50  0000 L CNN
-F 1 "4.7k" H 3459 805 50  0000 L CNN
-F 2 "Resistor_SMD:R_0603_1608Metric" H 3400 850 50  0001 C CNN
-F 3 "~" H 3400 850 50  0001 C CNN
-	1    3400 850
-	1    0    0    -1
-$EndComp
-$Comp
-L Device:R_Small R16
-U 1 1 5E89F635
-P 3250 850
-F 0 "R16" H 3100 900 50  0000 L CNN
-F 1 "4.7k" H 3050 800 50  0000 L CNN
-F 2 "Resistor_SMD:R_0603_1608Metric" H 3250 850 50  0001 C CNN
-F 3 "~" H 3250 850 50  0001 C CNN
-	1    3250 850
-	1    0    0    -1
-$EndComp
-Wire Wire Line
-	3250 950  3250 1200
-Wire Wire Line
-	3250 1200 3450 1200
-Wire Wire Line
-	3450 1200 3450 1350
-Connection ~ 3450 1350
-Wire Wire Line
-	3450 1350 4300 1350
-Wire Wire Line
-	3400 950  3400 1150
-Wire Wire Line
-	3400 1150 3500 1150
-Wire Wire Line
-	3500 1150 3500 1450
-Connection ~ 3500 1450
-Wire Wire Line
-	3500 1450 4300 1450
-Wire Wire Line
-	3250 750  3250 700
-Wire Wire Line
-	3250 700  3350 700
-Wire Wire Line
-	3400 700  3400 750
-Wire Wire Line
-	3350 700  3350 600
-Connection ~ 3350 700
-Wire Wire Line
-	3350 700  3400 700
-Text GLabel 3350 600  0    50   Input ~ 0
+	3350 1400 3450 1400
+Wire Wire Line
+	3350 1500 3500 1500
+Connection ~ 3450 1400
+Wire Wire Line
+	3450 1400 4300 1400
+Connection ~ 3500 1500
+Wire Wire Line
+	3500 1500 4300 1500
+Wire Wire Line
+	3250 750  3350 750
+Wire Wire Line
+	3350 750  3350 650
+Connection ~ 3350 750
+Text GLabel 3350 650  0    50   Input ~ 0
 +3.3V
 Wire Notes Line
@@
 Wire Wire Line
 	2450 4300 2350 4300
+$Comp
+L Device:R_Small R?
+U 1 1 5EAF962B
+P 3300 1000
+AR Path="/5EA28FED/5EAF962B" Ref="R?"  Part="1"
+AR Path="/5EA28FEB/5EAF962B" Ref="R?"  Part="1"
+F 0 "R?" H 3100 1050 50  0000 L CNN
+F 1 "4.7K" H 3050 950 50  0000 L CNN
+F 2 "Resistor_SMD:R_0603_1608Metric" H 3300 1000 50  0001 C CNN
+F 3 "~" H 3300 1000 50  0001 C CNN
+	1    3300 1000
+	1    0    0    -1
+$EndComp
+$Comp
+L Device:R_Small R?
+U 1 1 5EAFCD23
+P 3500 1000
+AR Path="/5EA28FED/5EAFCD23" Ref="R?"  Part="1"
+AR Path="/5EA28FEB/5EAFCD23" Ref="R?"  Part="1"
+F 0 "R?" H 3300 1050 50  0000 L CNN
+F 1 "4.7K" H 3250 950 50  0000 L CNN
+F 2 "Resistor_SMD:R_0603_1608Metric" H 3500 1000 50  0001 C CNN
+F 3 "~" H 3500 1000 50  0001 C CNN
+	1    3500 1000
+	-1   0    0    -1
+$EndComp
+Wire Wire Line
+	3450 1150 3300 1150
+Wire Wire Line
+	3300 1150 3300 1100
+Wire Wire Line
+	3450 1150 3450 1400
+Wire Wire Line
+	3500 1100 3500 1500
+Wire Wire Line
+	3500 900  3500 750
+Wire Wire Line
+	3350 750  3500 750
+Wire Wire Line
+	3300 900  3300 850
+Wire Wire Line
+	3300 850  3250 850
+Wire Wire Line
+	3250 850  3250 750
 $EndSCHEMATC

Commit message: Add files via upload
Parts:
- removed J3, J6: Conn_01x23, Connector_PinHeader_2.54mm:PinHeader_1x23_P2.54mm_Vertical, symbol Connector_Generic:Conn_01x23
- removed J7: Conn_02x02_Top_Bottom, Connector_PinHeader_2.54mm:PinHeader_2x02_P2.54mm_Vertical, symbol Connector_Generic:Conn_02x02_Top_Bottom
- removed R? (x2): 4.7K, Resistor_SMD:R_0603_1608Metric, symbol Device:R_Small
- added J3, J6: Conn_01x25, Connector_PinHeader_2.54mm:PinHeader_1x25_P2.54mm_Vertical, symbol Connector_Generic:Conn_01x25
- renumbered J4 to UART1
Connections:
- net +3.3V: now also J6.1 (Pin_1)
- net +5V: now also J3.1 (Pin_1)
- net GND: now also J3.2 (Pin_2), J6.2 (Pin_2)
- net PA0: now also J6.8 (Pin_8)
- net PA1: now also J6.9 (Pin_9)
- net PA10: now also J3.18 (Pin_18)
- net PA11: now also J3.17 (Pin_17)
- net PA12: now also J3.16 (Pin_16)
- net PA13: now also J3.15 (Pin_15); no longer UART1.2 (Pin_2)
- net PA14: now also J3.14 (Pin_14); no longer UART1.3 (Pin_3)
- net PA15: now also J3.13 (Pin_13)
- net PA2: now also J6.10 (Pin_10)
- net PA3: now also J6.11 (Pin_11)
- net PA4: now also J6.12 (Pin_12)
- net PA5: now also J6.13 (Pin_13)
- net PA6: now also J6.14 (Pin_14)
- net PA7: now also J6.15 (Pin_15)
- net PA8: now also J3.20 (Pin_20)
- net PA9: now also J3.19 (Pin_19)
- net PB0: now also J6.18 (Pin_18)
- net PB1: now also J6.19 (Pin_19)
- net PB11: now also J6.22 (Pin_22)
- net PB12: now also J6.23 (Pin_23)
- net PB13: now also J6.24 (Pin_24)
- net PB14: now also J6.25 (Pin_25)
- net PB15: now also J3.25 (Pin_25)
- net PB2: now also J6.20 (Pin_20)
- net PB3: now also J3.8 (Pin_8)
- net PB4: now also J3.7 (Pin_7)
- net PB5: now also J3.6 (Pin_6)
- net PB6: now also J3.5 (Pin_5)
- net PB7: now also J3.4 (Pin_4)
- net PB9: now also J3.3 (Pin_3)
- net PC0: now also J6.4 (Pin_4)
- net PC1: now also J6.5 (Pin_5)
- net PC10: now also J3.12 (Pin_12)
- net PC11: now also J3.11 (Pin_11)
- net PC12: now also J3.10 (Pin_10)
- net PC13: now also J6.3 (Pin_3)
- net PC2: now also J6.6 (Pin_6)
- net PC3: now also J6.7 (Pin_7)
- net PC4: now also UART1.2 (Pin_2), J6.16 (Pin_16)
- net PC5: now also UART1.3 (Pin_3), J6.17 (Pin_17)
- net PC6: now also J3.24 (Pin_24)
- net PC7: now also J3.23 (Pin_23)
- net PC8: now also J3.22 (Pin_22)
- net PC9: now also J3.21 (Pin_21)
- net PD2: now also J3.9 (Pin_9)
- new net PB10: J6.21 (Pin_21)
Other:
- note removed: "SWCLK"
- note removed: "SWDIO\n"
- moved on the sheet: C25, J5
