File: STM32G473RET6 Development Board/Dev_Pro.kicad_pcb (KiCad board)
At the start: 2 copper layers, 38.6 x 77.7 mm, 79 parts, among them IC1 STM32G473RET6, J1 Screw_Terminal_01x02, J2 USB_C_Receptacle_USB2.0, J3 Conn_01x23, J4 Conn_01x04, J5 Conn_01x04, J6 Conn_01x23, J7 Conn_02x02_Top_Bottom, J8 Conn_ARM_JTAG_SWD_10, P1 USB_C_Plug_USB2.0, Q1 DMP3013SFV, Q2 IRF9394M, Q3 IRF9394M, SW1 SW_SPST, SW2 SW_DIP_x02, U1 AP2127R-3.3, U2 INA260, U3 CP2102N-A01-GQFN24, U4 MPU-9250, Y1 Crystal_GND23, Y2 Crystal_GND23

Commit message: Add files via upload
Parts:
- removed F2: Fuse, Fuse:Fuse_0603_1608Metric
- removed Q1: DMP3013SFV, Package_SON:Diodes_PowerDI3333-8
- removed Q2, Q3: IRF9394M, Package_DirectFET:DirectFET_MC
- removed R16, R17: 4.7k, Resistor_SMD:R_0603_1608Metric
- removed SW2: SW_DIP_x02, Button_Switch_SMD:SW_DIP_SPSTx02_Slide_6.7x6.64mm_W8.61mm_P2.54mm_LowProfile
- added JP3: Jumper, Jumper:SolderJumper-2_P1.3mm_Open_Pad1.0x1.5mm, F.Cu at (123.1, 110.1)
- added JP4: Jumper, Jumper:SolderJumper-2_P1.3mm_Open_Pad1.0x1.5mm, F.Cu at (116.7, 117.6)
- added U5: IRF7205TRPB, Package_SO:SOP-8_3.9x4.9mm_P1.27mm, F.Cu at (82.5, 68.5)
- added U6: IRF7205TRPB, Package_SO:SOP-8_3.9x4.9mm_P1.27mm, F.Cu at (82.5, 74.9)
- added U7: IRF7205TRPB, Package_SO:SOP-8_3.9x4.9mm_P1.27mm, F.Cu at (90.9, 68.5)
- C1, C15, C18, C19, C2, C20, C21, C22, C23, C26, C27, C28, D1, FB1, R1, R10, R11, R12, R13: moved to B.Cu
- JP1: footprint Button_Switch_SMD:SW_DIP_SPSTx02_Slide_Copal_CHS-02A_W5.08mm_P1.27mm_JPin -> Jumper:SolderJumper-3_P1.3mm_Open_Pad1.0x1.5mm_NumberLabels
- JP2: footprint Button_Switch_SMD:SW_DIP_SPSTx02_Slide_Copal_CHS-02A_W5.08mm_P1.27mm_JPin -> Jumper:SolderJumper-3_P1.3mm_Open_Pad1.0x1.5mm
- moved R20 216.7 mm to (231.5, 32.5), turned to 90 degrees
- moved R19 212.7 mm to (223.5, 33.8), turned to 90 degrees
- moved C1 207.6 mm to (6.49, 72.8), turned to 180 degrees
- moved D1 207.2 mm to (4.25, 72.3), turned to 270 degrees
- moved FB1 204.4 mm to (6.88, 71.2), turned to 180 degrees
- moved C2 202.7 mm to (10.5, 64.8), turned to 180 degrees
- moved U1 197.4 mm to (8.90, 69.1), turned to 180 degrees
- moved C18 190.3 mm to (18.8, 12.0)
- moved C19 188.7 mm to (18.8, 10.8)
- moved R11 185.3 mm to (14.8, 11.5), turned to 180 degrees
- moved C21 184.7 mm to (20.5, 14.8), turned to 270 degrees
- moved C26 184.4 mm to (16.5, 59.0), turned to 90 degrees
- moved C20 183.9 mm to (21.8, 14.8), turned to 270 degrees
- moved C23 183.1 mm to (24.2, 14.8), turned to 270 degrees
- moved R10 182.5 mm to (11.5, 15.0), turned to 180 degrees
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Connections:
- net Net-(D2-Pad3) renamed /USB_to_UART/D-
- net Net-(D2-Pad4) renamed /USB_to_UART/D+
- C15 pad 2: /MCU/NRST -> NRST
- D4 pad 1: PC5 -> PC4
- IC1 pad 60: PB7 -> +3.3V
- IC1 pad 61: PB8 -> +3.3V
- IC1 pad 7: /MCU/NRST -> NRST
- J3 pad 12: PB7 -> +3.3V
- J3 pad 13: PB8 -> +3.3V
- J5 pad 2: PB7 -> +3.3V
- J5 pad 3: PB8 -> +3.3V
- R1 pad 1: /MCU/NRST -> NRST
- R2 pad 1: /USB Power Delivery/VBUS -> Net-(R2-Pad1)
- R2 pad 2: Net-(Q2-Pad1) -> /USB Power Delivery/VBUS
- R4 pad 2: PB8 -> +3.3V
- R5 pad 2: PB7 -> +3.3V
- SW1 pad 1: /MCU/NRST -> NRST
- U2 pad 1: Net-(Q2-Pad1) -> Net-(R2-Pad1)
- U2 pad 2: Net-(Q2-Pad1) -> Net-(R2-Pad1)
- U2 pad 3: Net-(Q2-Pad1) -> Net-(R2-Pad1)
- U2 pad 8: PB7 -> +3.3V
- U2 pad 9: PB8 -> +3.3V
Routing:
- net +3.3V: track 15.7 -> 49.2 mm, vias 0 -> 10
- net +5V: track 0.00 -> 21.7 mm, vias 0 -> 2
- net /USB_to_UART/D+: track 0.00 -> 13.6 mm
- net NRST: track 0.00 -> 12.7 mm, vias 0 -> 1
- net /USB_to_UART/D-: track 0.00 -> 12.4 mm
- net Net-(D2-Pad2): track 0.00 -> 11.8 mm, vias 0 -> 2
- net /MCU/OSC8_IN: track 0.00 -> 7.83 mm
- net Net-(C1-Pad1): track 0.00 -> 7.34 mm, vias 0 -> 1
- net Net-(D4-Pad2): track 0.00 -> 5.33 mm, vias 0 -> 1
- net PC4: track 0.00 -> 5.11 mm
- net /MCU/OSC8_OUT: track 0.00 -> 4.13 mm
- net Net-(C10-Pad1): track 0.00 -> 3.96 mm
- net Net-(C12-Pad1): track 0.00 -> 3.49 mm
- net Net-(D3-Pad2): track 0.00 -> 3.25 mm, vias 0 -> 1
- net PA4: track 0.00 -> 3.07 mm
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Other:
- board size 38.6 x 77.7 mm -> 33 x 80 mm
- net class Power added: clearance 0.2, trace_width 2.76552, via_dia 0.8, via_drill 0.4
- rule trace_min: 0.2 -> 0.1524

Commit message: Add files via upload
Parts:
- removed C26, C27, C28: C_Small, Capacitor_SMD:C_0402_1005Metric
- removed D5: LED, LED_SMD:LED_0805_2012Metric_Pad1.15x1.40mm_HandSolder
- removed J7: Conn_02x02_Top_Bottom, Connector_PinHeader_2.54mm:PinHeader_2x02_P2.54mm_Vertical
- removed JP1: ADDR A1, Jumper:SolderJumper-3_P1.3mm_Open_Pad1.0x1.5mm_NumberLabels
- removed JP2: ADDR A0, Jumper:SolderJumper-3_P1.3mm_Open_Pad1.0x1.5mm
- removed JP3, JP4: Jumper, Jumper:SolderJumper-2_P1.3mm_Open_Pad1.0x1.5mm
- removed R14: 22.1K, Resistor_SMD:R_0603_1608Metric
- removed R15: 47.5K, Resistor_SMD:R_0603_1608Metric
- removed R18, R8, R9: R_Small, Resistor_SMD:R_0603_1608Metric
- removed U2: INA260, Package_SO:TSSOP-16_4.4x5mm_P0.65mm
- removed U4: MPU-9250, Sensor_Motion:InvenSense_QFN-24_3x3mm_P0.4mm
- removed U5, U7: IRF7205TRPB, Package_SO:SOP-8_3.9x4.9mm_P1.27mm
- added C29: C, Capacitor_SMD:CP_Elec_3x5.3, F.Cu at (156.0, 66.8)
- added C30: C, Capacitor_SMD:CP_Elec_3x5.3, F.Cu at (139.8, 66.5)
- C1, C15, C2, D1, FB1, R1, R12, R13: moved to F.Cu
- C13, C14, C16, C17, C24, C3, C4, C5, C6, C7, C8, D2, F1, R6, R7, U3, U6: moved to B.Cu
- J3, J6: value Conn_01x23 -> Conn_01x25; footprint Connector_PinHeader_2.54mm:PinHeader_1x23_P2.54mm_Vertical -> Connector_PinHeader_2.54mm:PinHeader_1x25_P2.54mm_Vertical
- R2: value R -> R_Small
- R3, R4, R5: value 4.7K -> R_Small
- moved P1 196.6 mm to (148.5, 148.2), turned to 0 degrees
- moved I2C 190.6 mm to (159.5, 146.2), turned to 0 degrees
- moved UART1 187.6 mm to (131.5, 146.2), turned to 0 degrees
- moved D2 184.5 mm to (151.9, 140.7), turned to 180 degrees
- moved R10 178.3 mm to (148.0, 129.8), turned to 90 degrees
- moved U3 178.0 mm to (148.5, 135.0), turned to 90 degrees
- moved C21 177.5 mm to (146.5, 139.8)
- moved R11 177.2 mm to (144.0, 132.8)
- moved C19 176.6 mm to (142.0, 137.2), turned to 180 degrees
- moved C20 175.7 mm to (145.2, 139.8)
- moved C18 174.8 mm to (142.0, 136.0), turned to 180 degrees
- moved C23 172.4 mm to (144.5, 138.2), turned to 180 degrees
- moved C22 172.4 mm to (144.5, 137.0), turned to 180 degrees
- moved D4 165.1 mm to (130.8, 142.5), turned to 180 degrees
- moved D3 164.9 mm to (130.8, 140.0), turned to 180 degrees
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- renumbered Y1 to 32KHz, Y2 to 8MHz, J5 to I2C, SW1 to RESET, J8 to SWD, J4 to UART1
Connections:
- I2C pad 2: +3.3V -> PB7
- I2C pad 3: +3.3V -> PB8
- IC1 pad 30: /MCU/PB10 -> PB10
- IC1 pad 60: +3.3V -> PB7
- IC1 pad 61: +3.3V -> PB8
- J2 pad A4: /USB Power Delivery/VBUS -> Net-(C29-Pad2)
- J2 pad A5: PB6 -> Net-(J2-PadA5)
- J2 pad A9: /USB Power Delivery/VBUS -> Net-(C29-Pad2)
- J2 pad B4: /USB Power Delivery/VBUS -> Net-(C29-Pad2)
- J2 pad B5: PB4 -> Net-(J2-PadB5)
- J2 pad B9: /USB Power Delivery/VBUS -> Net-(C29-Pad2)
- J3 pad 1: PA13 -> +5V
- J3 pad 10: PB5 -> PC12
- J3 pad 11: PB6 -> PC11
- J3 pad 12: +3.3V -> PC10
- J3 pad 13: +3.3V -> PA15
- J3 pad 14: PB9 -> PA14
- J3 pad 15: PA12 -> PA13
- J3 pad 16: PA11 -> PA12
- J3 pad 17: PA10 -> PA11
- J3 pad 18: PA9 -> PA10
- J3 pad 19: PA8 -> PA9
- J3 pad 2: PA14 -> GND
- J3 pad 20: PC9 -> PA8
- J3 pad 21: PC8 -> PC9
- J3 pad 22: PC7 -> PC8
- J3 pad 23: PC6 -> PC7
- J3 pad 3: PA15 -> PB9
- J3 pad 4: PC10 -> PB7
- J3 pad 5: PC11 -> PB6
- J3 pad 6: PC12 -> PB5
- J3 pad 7: PD2 -> PB4
- J3 pad 9: PB4 -> PD2
- J6 pad 1: PC13 -> +3.3V
- J6 pad 10: PA4 -> PA2
- J6 pad 11: PA5 -> PA3
- J6 pad 12: PA6 -> PA4
- J6 pad 13: PA7 -> PA5
- J6 pad 14: PC4 -> PA6
- J6 pad 15: PC5 -> PA7
- J6 pad 16: PB0 -> PC4
- J6 pad 17: PB1 -> PC5
- J6 pad 18: PB2 -> PB0
- J6 pad 19: PB11 -> PB1
- J6 pad 2: PC0 -> GND
- J6 pad 20: PB12 -> PB2
- J6 pad 21: PB13 -> PB10
- J6 pad 22: PB14 -> PB11
- J6 pad 23: PB15 -> PB12
- J6 pad 3: PC1 -> PC13
- J6 pad 4: PC2 -> PC0
- J6 pad 5: PC3 -> PC1
- J6 pad 6: PA0 -> PC2
- J6 pad 7: PA1 -> PC3
- J6 pad 8: PA2 -> PA0
- J6 pad 9: PA3 -> PA1
- R2 pad 1: Net-(R2-Pad1) -> PB6
- R2 pad 2: /USB Power Delivery/VBUS -> Net-(J2-PadA5)
- R3 pad 1: +3.3V -> PB4
- R3 pad 2: Net-(R3-Pad2) -> Net-(J2-PadB5)
- R4 pad 1: +3.3V -> PA11
- R4 pad 2: +3.3V -> /USB Power Delivery/DA-
- R5 pad 1: +3.3V -> PA12
- R5 pad 2: +3.3V -> /USB Power Delivery/DA+
- R6 pad 1: /USB Power Delivery/VBUS -> Net-(F1-Pad1)
- U6 pad 1: Net-(F1-Pad1) -> Net-(C29-Pad2)
- U6 pad 2: Net-(F1-Pad1) -> Net-(C29-Pad2)
- U6 pad 3: Net-(F1-Pad1) -> Net-(C29-Pad2)
- U6 pad 5: /USB Power Delivery/VBUS -> Net-(F1-Pad1)
- U6 pad 6: (no net) -> Net-(F1-Pad1)
- U6 pad 7: /USB Power Delivery/VBUS -> Net-(F1-Pad1)
- U6 pad 8: /USB Power Delivery/VBUS -> Net-(F1-Pad1)
- UART1 pad 2: PA13 -> PC4
- UART1 pad 3: PA14 -> PC5
Routing:
- net GND: track 0.00 -> 330.2 mm, vias 0 -> 3
- net +3.3V: track 49.2 -> 221.6 mm, vias 10 -> 5
- net +5V: track 21.7 -> 130.7 mm, vias 2 -> 3
- net PC5: track 2.66 -> 81.0 mm, vias 0 -> 1
- net PB7: track 0.00 -> 75.1 mm, vias 0 -> 1
- net PA13: track 0.00 -> 72.9 mm, vias 0 -> 1
- net PC4: track 5.11 -> 75.9 mm
- net PA10: track 0.00 -> 63.8 mm
- net PA14: track 0.00 -> 63.6 mm, vias 0 -> 1
- net PA12: track 0.00 -> 62.1 mm, vias 0 -> 1
- net NRST: track 12.7 -> 74.7 mm, vias 1 -> 0
- net PA11: track 0.00 -> 52.8 mm
- net PB8: track 0.00 -> 51.5 mm, vias 0 -> 1
- net PB3: track 0.00 -> 50.9 mm, vias 0 -> 1
- net PB4: track 0.00 -> 49.7 mm, vias 0 -> 1
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- added copper zone on B.Cu, net GND
- added copper zone on F.Cu, net GND
Other:
- board size 33 x 80 mm -> 40 x 90 mm
- board text added: "+3.3V"
- board text added: "+5V"
- board text added: "GND"
- board text added: "PA0"
- board text added: "PA1"
- board text added: "PA10"
- board text added: "PA11"
- board text added: "PA12"
- board text added: "PA13"
- board text added: "PA14"
- board text added: "PA15"
- board text added: "PA2"
- board text added: "PA3"
- board text added: "PA4"
- board text added: "PA5"
- board text added: "PA6"
- board text added: "PA7"
- board text added: "PA8"
- board text added: "PA9"
- board text added: "PB0"
- board text added: "PB1"
- board text added: "PB10"
- board text added: "PB12"
- board text added: "PB13"
- board text added: "PB14"
- board text added: "PB15"
- board text added: "PB2"
- board text added: "PB3"
- board text added: "PB4"
- board text added: "PB5"
- board text added: "PB6"
- board text added: "PB7"
- board text added: "PB9"
- board text added: "PC0"
- board text added: "PC1"
- board text added: "PC10"
- board text added: "PC11"
- board text added: "PC12"
- board text added: "PC13"
- board text added: "PC2"
- board text added: "PC4"
- board text added: "PC5"
- board text added: "PC6"
- board text added: "PC7"
- board text added: "PC8"
- board text added: "PC9"
- board text added: "PD2"
- board text added: "POWER"
- board text added: "STM32G473RET6"
