File: STM32G473RET6 Development Board/MCU.sch (KiCad schematic (older format))
At the start: 11 parts

Commit message: Add files via upload
Parts:
- added C? (x5): 100N, symbol Device:C_Small
- added R?: R_Small, symbol Device:R_Small
- added SW?: SW_SPST, symbol Switch:SW_SPST
- added Y? (x2): Crystal_GND23, symbol Device:Crystal_GND23
Connections:
- net labels added: PB8
- net labels removed: BOOT0
- wire segments 115 -> 159
Other:
- moved on the sheet: C?, IC?

Commit message: Add files via upload
Parts:
- added R19, R20: R_Small, Resistor_SMD:R_0603_1608Metric, symbol Device:R_Small
- C10, C11, C12, C13, C14, C15, C16, C17, C3, C4, C5, C6, C7, C8, C9: renamed from C?; footprint (none) -> Capacitor_SMD:C_0402_1005Metric
- IC1: renamed from IC?; footprint QFP50P1200X1200X160-64N -> ASSETS:QFP50P1200X1200X160-64N_STM32G473RET6
- R1: renamed from R?; footprint (none) -> Resistor_SMD:R_0603_1608Metric
- SW1: renamed from SW?; footprint (none) -> Button_Switch_SMD:SW_SPST_TL3342
- Y1, Y2: renamed from Y?; footprint (none) -> Crystal:Crystal_SMD_SeikoEpson_FA238-4Pin_3.2x2.5mm
Connections:
- net OSC32_OUT: now also R19.1; no longer C10.1, Y1.4
- net OSC8_OUT: now also R20.1; no longer C12.1, Y2.4
- new net: C10.1, R19.2, Y1.4
- new net: C12.1, R20.2, Y2.4

Commit message: Add files via upload
Changed lines of the file:
@@
 Wire Wire Line
 	2950 4300 2950 4550
-Text Label 2950 4550 3    50   ~ 0
-PB10
 Wire Wire Line
 	3450 3200 3700 3200
@@
 Wire Wire Line
 	5700 4100 5600 4100
-Text Label 5700 3800 1    50   ~ 0
-NRST
 Text GLabel 5050 4100 0    50   Input ~ 0
 +3.3V
@@
 Wire Wire Line
 	6850 3150 6650 3150
+Text GLabel 5700 3800 0    50   Input ~ 0
+NRST
+Text GLabel 2950 4550 3    50   Input ~ 0
+PB10
 $EndSCHEMATC

Commit message: Add files via upload
Changed lines of the file:
@@
 $Descr User 7874 7874
 encoding utf-8
-Sheet 3 7
+Sheet 3 6
 Title "STM32G473RETx "
 Date ""
@@
 Wire Wire Line
 	2850 4450 2800 4450
-Wire Wire Line
-	1950 950  1950 1200
 Wire Wire Line
 	1850 950  1850 1200
@@
 Wire Wire Line
 	2200 6600 2400 6600
-Text Label 3500 2300 0    50   ~ 0
-D+
-Text Label 3500 2400 0    50   ~ 0
-D-
 Text GLabel 1200 1700 1    50   Input ~ 0
 +3.3V
@@
 Text GLabel 2050 950  1    50   Input ~ 0
 PB7
-Text GLabel 1950 950  1    50   Input ~ 0
-PB8
 Text GLabel 1850 950  1    50   Input ~ 0
 PB9
@@
 Text GLabel 2950 4550 3    50   Input ~ 0
 PB10
+Wire Wire Line
+	1950 700  2100 700
+Wire Wire Line
+	2100 700  2100 650
+Wire Wire Line
+	1950 700  1950 1200
+Text GLabel 2100 650  2    50   Input ~ 0
+PB8
 $EndSCHEMATC
