File: STM32G473RET6 Development Board/USB Power Delivery.sch (KiCad schematic (older format))
At the start: 5 parts

Commit message: Add files via upload
Parts:
- added F? (x2): Fuse, symbol Device:Fuse
- added J?: Screw_Terminal_01x02, symbol Connector:Screw_Terminal_01x02
- added Q?: DMP3013SFV, Package_SON:Diodes_PowerDI3333-8, symbol Transistor_FET:DMP3013SFV
- added Q? (x2): IRF9394M, Package_DirectFET:DirectFET_MC, symbol Transistor_FET:IRF9394M
- added R? (x4): R_Small, symbol Device:R_Small
- added R?: R, symbol Device:R
Connections:
- net GND: now also J?.1 (Pin_1), R?.2
- net PA10: now also Q?.4 (G)
- net PA11: now also Q?.2 (G), Q?.2 (G), R?.1; no longer J?.A7 (DA-), J?.B7 (DB-)
- net PA12: now also R?.1; no longer J?.A6 (DA+), J?.B6 (DB+)
- net VBUS: now also Q?.1 (S), Q?.2 (S), Q?.3 (S), R?.1, R?.1
- net CC1 renamed PB6
- net CC2 renamed PB4
- new net: F?.2, F?.2, J?.2 (Pin_2)
- new net: F?.1, Q?.5 (D)
- new net: F?.1, Q?.1 (D)
- new net: Q?.3 (S), Q?.3 (S)
- new net: Q?.1 (D), R?.2
- new net DA+: J?.A6 (DA+), J?.B6 (DB+), R?.2
- new net DA-: J?.A7 (DA-), J?.B7 (DB-), R?.2
- new net PA0: R?.1, R?.2
Other:
- moved on the sheet: J?, JP?, Q?

Commit message: Add files via upload
Parts:
- removed J?: 12401610E4#2A, ASSETS:USB_C_Receptacle_HRO_TYPE-C-31-M-12, symbol K_USB_C_receptacle:12401610E4#2A
- removed JP? (x2): Jumper, symbol Device:Jumper
- removed Q? (x2): DMN10H700S, Package_TO_SOT_SMD:SOT-23, symbol Transistor_FET:DMN10H700S
- added J2: USB_C_Receptacle_USB2.0, ASSETS:USB_C_Receptacle_HRO_TYPE-C-31-M-12, symbol Connector:USB_C_Receptacle_USB2.0
- added JP1: ADDR A1, Button_Switch_SMD:SW_DIP_SPSTx02_Slide_Copal_CHS-02A_W5.08mm_P1.27mm_JPin, symbol Device:Jumper_NC_Dual
- added JP2: ADDR A0, Button_Switch_SMD:SW_DIP_SPSTx02_Slide_Copal_CHS-02A_W5.08mm_P1.27mm_JPin, symbol Device:Jumper_NC_Dual
- added R3, R4, R5: 4.7K, Resistor_SMD:R_0603_1608Metric, symbol Device:R_Small
- added SW2: SW_DIP_x02, Button_Switch_SMD:SW_DIP_SPSTx02_Slide_6.7x6.64mm_W8.61mm_P2.54mm_LowProfile, symbol Switch:SW_DIP_x02
- added U2: INA260, Package_SO:TSSOP-16_4.4x5mm_P0.65mm, symbol Sensor:INA260
- F1, F2: renamed from F?; footprint (none) -> Fuse:Fuse_0603_1608Metric
- J1: renamed from J?; footprint (none) -> Connector_JST:JST_EH_S2B-EH_1x02_P2.50mm_Horizontal
- R2, R6, R7, R8, R9: renamed from R?; footprint (none) -> Resistor_SMD:R_0603_1608Metric
- gave numbers to parts that had none: 3
Connections:
- net DA+: now also J2.A6 (D+), J2.B6 (D+)
- net DA-: now also J2.A7 (D-), J2.B7 (D-)
- net GND: now also J2.A1 (GND), J2.A12 (GND), J2.B1 (GND), J2.B12 (GND), J2.S1 (SHIELD), JP1.3, JP2.3, SW2.1, SW2.2, U2.11 (GND), U2.6 (GND)
- net PA10: now also SW2.3
- net PA9: now also SW2.4
- net PB4: now also J2.B5 (CC2)
- net PB6: now also J2.A5 (CC1)
- net VBUS: now also J2.A4 (VBUS), J2.A9 (VBUS), J2.B4 (VBUS), J2.B9 (VBUS), U2.14 (IN-), U2.15 (IN-), U2.16 (IN-)
- net at Q2.1 (D), R2.2: now also U2.1 (IN+), U2.2 (IN+), U2.3 (IN+)
- new net: JP1.2, U2.4 (A1)
- new net: JP2.2, U2.5 (A0)
- new net: R3.2, U2.7 (ALERT)
- new net +3.3V: JP1.1, JP2.1, R3.1, R4.1, R5.1, U2.10 (VS)
- new net PB7: R5.2, U2.8 (SDA)
- new net PB8: R4.2, U2.9 (SCL)
- no-connect marks 10 -> 2
Other:
- note added: "SCL\n"
- note added: "SDA"
- moved on the sheet: Q2, Q3, R2, R8, R9

Commit message: Add files via upload
Parts:
- removed F2: Fuse, Fuse:Fuse_0603_1608Metric, symbol Device:Fuse
- removed JP1: ADDR A1, Button_Switch_SMD:SW_DIP_SPSTx02_Slide_Copal_CHS-02A_W5.08mm_P1.27mm_JPin, symbol Device:Jumper_NC_Dual
- removed JP2: ADDR A0, Button_Switch_SMD:SW_DIP_SPSTx02_Slide_Copal_CHS-02A_W5.08mm_P1.27mm_JPin, symbol Device:Jumper_NC_Dual
- removed Q1: DMP3013SFV, Package_SON:Diodes_PowerDI3333-8, symbol Transistor_FET:DMP3013SFV
- removed Q2, Q3: IRF9394M, Package_DirectFET:DirectFET_MC, symbol Transistor_FET:IRF9394M
- removed R2: R, Resistor_SMD:R_0603_1608Metric, symbol Device:R
- removed R8, R9: R_Small, Resistor_SMD:R_0603_1608Metric, symbol Device:R_Small
- removed SW2: SW_DIP_x02, Button_Switch_SMD:SW_DIP_SPSTx02_Slide_6.7x6.64mm_W8.61mm_P2.54mm_LowProfile, symbol Switch:SW_DIP_x02
- removed U2: INA260, Package_SO:TSSOP-16_4.4x5mm_P0.65mm, symbol Sensor:INA260
- added C29, C30: C, Capacitor_SMD:CP_Elec_3x5.3, symbol Device:C
- added R2: R_Small, Resistor_SMD:R_0603_1608Metric, symbol Device:R_Small
- added U6: IRF7205TRPB, Package_SO:SOP-8_3.9x4.9mm_P1.27mm, symbol Transistor_FET:IRF7205TRPB
- R3, R4, R5: value 4.7K -> R_Small
Connections:
- net PB7 is gone; now on net DA+: R5.2
- net PB8 is gone; now on net DA-: R4.2
- net GND: now also C29.1, C30.1
- net PA10: now also U6.4 (G)
- net PA11: now also R4.1
- net PA12: now also R5.1
- net PB4: now also R3.1; no longer J2.B5 (CC2)
- net PB6: now also R2.1; no longer J2.A5 (CC1)
- net at F1.2, J1.2 (Pin_2): now also C30.2
- net at F1.1: now also R6.1, U6.5 (D), U6.6 (D), U6.7 (D), U6.8 (D)
- net at R3.2: now also J2.B5 (CC2)
- removed net +3.3V: R3.1, R4.1, R5.1
- net VBUS: no longer names the net of J2.A4 (VBUS), J2.A9 (VBUS), J2.B4 (VBUS), J2.B9 (VBUS)
- net VBUS: now also C29.2, U6.1 (S), U6.2 (S), U6.3 (S); no longer R6.1
- new net: J2.A5 (CC1), R2.2
Other:
- note removed: "SCL\n"
- note removed: "SDA"
- moved on the sheet: F1, J1, R6, R7

Commit message: Add files via upload
Changed lines of the file:
@@
 $Descr User 7874 7874
 encoding utf-8
-Sheet 4 7
+Sheet 4 6
 Title ""
 Date ""
@@
 	0    1    -1   0
 $EndComp
-Wire Wire Line
-	2950 3700 3200 3700
 $Comp
 L Device:R_Small R4
@@
 	0    1    -1   0
 $EndComp
-Wire Wire Line
-	2950 3500 3200 3500
 Text Label 2550 3700 0    50   ~ 0
 DA+
 Text Label 2500 3500 0    50   ~ 0
 DA-
-Text GLabel 3200 3700 2    50   Input ~ 0
+Text GLabel 3400 3700 2    50   Input ~ 0
 PA12
-Text GLabel 3200 3500 2    50   Input ~ 0
+Text GLabel 3400 3500 2    50   Input ~ 0
 PA11
 Text GLabel 2500 3150 2    50   Input ~ 0
@@
 Wire Wire Line
 	2200 3250 2150 3250
+Wire Wire Line
+	2950 3500 3400 3500
+Wire Wire Line
+	2950 3700 3400 3700
 $EndSCHEMATC
