File: STM32G473RET6 Development Board/USB_to_UART.sch (KiCad schematic (older format))
At the start: 0 parts

Commit message: Add files via upload
Parts:
- added C? (x3): 0.1U, symbol Device:C_Small
- added C? (x3): 4.7U, symbol Device:C_Small
- added D? (x2): LED, symbol Device:LED
- added D?: SP0503BAHT, Package_TO_SOT_SMD:SOT-143, symbol Power_Protection:SP0503BAHT
- added P?: USB_C_Plug_USB2.0, symbol Connector:USB_C_Plug_USB2.0
- added R? (x4): 1K, symbol Device:R_Small
- added R?: 22.1K, symbol Device:R_Small
- added R?: 47.5K, symbol Device:R_Small
- added U?: CP2102N-A01-GQFN24, Package_DFN_QFN:QFN-24-1EP_4x4mm_P0.5mm_EP2.6x2.6mm, symbol Interface_USB:CP2102N-A01-GQFN24
Connections:
- new net: D?.2 (A), R?.2 (x2)
- new net: R?.1, U?.15 (~SUSPENDb)
- new net: D?.4 (K), P?.A6 (D+), U?.3 (D+)
- new net: D?.3 (K), P?.A7 (D-), U?.4 (D-)
- new net: D?.2 (K), P?.A4 (VBUS), P?.A9 (VBUS), P?.B4 (VBUS), P?.B5 (VCONN), P?.B9 (VBUS), U?.8 (VBUS)
- new net: R?.2, U?.9 (~RSTb)
- new net +3.3V: C?.1, C?.1, C?.1, C?.1, R?.1, U?.5 (VIO), U?.6 (VDD)
- new net +3.3v: R?.1, R?.1
- new net +5V: C?.1, C?.1, R?.1, U?.7 (REGIN)
- new net GND: C?.2, C?.2, C?.2, C?.2, C?.2, C?.2, D?.1 (A), P?.A1 (GND), P?.A12 (GND), P?.B1 (GND), P?.B12 (GND), P?.S1 (SHIELD), R?.2, R?.2, U?.2 (GND), U?.25 (GND)
- new net IO: R?.1, R?.2
- new net RXD: U?.20 (RXD)
- new net TXD: D?.1 (K), D?.1 (K), U?.21 (TXD)
- no-connect marks 0 -> 13

Commit message: Add files via upload
Parts:
- C18, C19, C20, C21, C22, C23: renamed from C?; footprint (none) -> Capacitor_SMD:C_0402_1005Metric
- D3, D4: renamed from D?; footprint (none) -> LED_SMD:LED_0805_2012Metric_Pad1.15x1.40mm_HandSolder
- P1: renamed from P?; footprint (none) -> ASSETS:USB_C_Receptacle_HRO_TYPE-C-31-M-12
- R10, R11, R12, R13, R14, R15: renamed from R?; footprint (none) -> Resistor_SMD:R_0603_1608Metric
- gave numbers to parts that had none: 2
Connections:
- net +3.3v is gone; now on net +3.3V: R12.1, R13.1
- net RXD renamed PC4
- net TXD renamed PC5
Changed lines of the file:
@@
 $EndDescr
 $Comp
-L Interface_USB:CP2102N-A01-GQFN24 U?
+L Interface_USB:CP2102N-A01-GQFN24 U3
 U 1 1 5E8893F1
 P 4350 4000
-F 0 "U?" H 4700 5000 50  0000 C CNN
+F 0 "U3" H 4700 5000 50  0000 C CNN
 F 1 "CP2102N-A01-GQFN24" H 4850 4850 50  0000 C CNN
 F 2 "Package_DFN_QFN:QFN-24-1EP_4x4mm_P0.5mm_EP2.6x2.6mm" H 4800 3200 50  0001 L CNN
@@
 $EndComp
 $Comp
-L Device:R_Small R?
+L Device:R_Small R11
 U 1 1 5E8899EA
 P 3400 3150
-F 0 "R?" H 3459 3196 50  0000 L CNN
+F 0 "R11" H 3459 3196 50  0000 L CNN
 F 1 "1K" H 3459 3105 50  0000 L CNN
-F 2 "" H 3400 3150 50  0001 C CNN
+F 2 "Resistor_SMD:R_0603_1608Metric" H 3400 3150 50  0001 C CNN
 F 3 "~" H 3400 3150 50  0001 C CNN
 	1    3400 3150
@@
 REGIN
 $Comp
-L Device:C_Small C?
+L Device:C_Small C19
 U 1 1 5E88A60E
 P 3150 1050
-F 0 "C?" H 3242 1096 50  0000 L CNN
+F 0 "C19" H 3242 1096 50  0000 L CNN
 F 1 "0.1U" H 3242 1005 50  0000 L CNN
-F 2 "" H 3150 1050 50  0001 C CNN
+F 2 "Capacitor_SMD:C_0402_1005Metric" H 3150 1050 50  0001 C CNN
 F 3 "~" H 3150 1050 50  0001 C CNN
 	1    3150 1050
@@
 $EndComp
 $Comp
-L Device:C_Small C?
+L Device:C_Small C18
 U 1 1 5E88B0C4
 P 2800 1050
-F 0 "C?" H 2600 1100 50  0000 L CNN
+F 0 "C18" H 2600 1100 50  0000 L CNN
 F 1 "4.7U" H 2400 1000 50  0000 L CNN
-F 2 "" H 2800 1050 50  0001 C CNN
+F 2 "Capacitor_SMD:C_0402_1005Metric" H 2800 1050 50  0001 C CNN
 F 3 "~" H 2800 1050 50  0001 C CNN
 	1    2800 1050
@@
 	2950 1300 2800 1300
 $Comp
-L power:GND #PWR?
+L power:GND #PWR0133
 U 1 1 5E88C3F3
 P 2950 1450
-F 0 "#PWR?" H 2950 1200 50  0001 C CNN
+F 0 "#PWR0133" H 2950 1200 50  0001 C CNN
 F 1 "GND" H 2955 1277 50  0000 C CNN
 F 2 "" H 2950 1450 50  0001 C CNN
@@
 VDD
 $Comp
-L Device:C_Small C?
+L Device:C_Small C21
 U 1 1 5E88E5FF
 P 4250 1050
-F 0 "C?" H 4342 1096 50  0000 L CNN
+F 0 "C21" H 4342 1096 50  0000 L CNN
 F 1 "0.1U" H 4342 1005 50  0000 L CNN
-F 2 "" H 4250 1050 50  0001 C CNN
+F 2 "Capacitor_SMD:C_0402_1005Metric" H 4250 1050 50  0001 C CNN
 F 3 "~" H 4250 1050 50  0001 C CNN
 	1    4250 1050
@@
 $EndComp
 $Comp
-L Device:C_Small C?
+L Device:C_Small C20
 U 1 1 5E88E605
 P 3900 1050
-F 0 "C?" H 3700 1100 50  0000 L CNN
+F 0 "C20" H 3700 1100 50  0000 L CNN
 F 1 "4.7U" H 3500 1000 50  0000 L CNN
-F 2 "" H 3900 1050 50  0001 C CNN
+F 2 "Capacitor_SMD:C_0402_1005Metric" H 3900 1050 50  0001 C CNN
 F 3 "~" H 3900 1050 50  0001 C CNN
 	1    3900 1050
@@
 	4050 1300 3900 1300
 $Comp
-L power:GND #PWR?
+L power:GND #PWR0134
 U 1 1 5E88E619
 P 4050 1450
-F 0 "#PWR?" H 4050 1200 50  0001 C CNN
+F 0 "#PWR0134" H 4050 1200 50  0001 C CNN
 F 1 "GND" H 4055 1277 50  0000 C CNN
 F 2 "" H 4050 1450 50  0001 C CNN
@@
 VIO
 $Comp
-L Device:C_Small C?
+L Device:C_Small C23
 U 1 1 5E88FDF3
 P 5350 1050
-F 0 "C?" H 5442 1096 50  0000 L CNN
+F 0 "C23" H 5442 1096 50  0000 L CNN
 F 1 "0.1U" H 5442 1005 50  0000 L CNN
-F 2 "" H 5350 1050 50  0001 C CNN
+F 2 "Capacitor_SMD:C_0402_1005Metric" H 5350 1050 50  0001 C CNN
 F 3 "~" H 5350 1050 50  0001 C CNN
 	1    5350 1050
@@
 $EndComp
 $Comp
-L Device:C_Small C?
+L Device:C_Small C22
 U 1 1 5E88FDF9
 P 5000 1050
-F 0 "C?" H 4800 1100 50  0000 L CNN
+F 0 "C22" H 4800 1100 50  0000 L CNN
 F 1 "4.7U" H 4600 1000 50  0000 L CNN
-F 2 "" H 5000 1050 50  0001 C CNN
+F 2 "Capacitor_SMD:C_0402_1005Metric" H 5000 1050 50  0001 C CNN
 F 3 "~" H 5000 1050 50  0001 C CNN
 	1    5000 1050
@@
 	5150 1300 5000 1300
 $Comp
-L power:GND #PWR?
+L power:GND #PWR0135
 U 1 1 5E88FE0D
 P 5150 1450
-F 0 "#PWR?" H 5150 1200 50  0001 C CNN
+F 0 "#PWR0135" H 5150 1200 50  0001 C CNN
 F 1 "GND" H 5155 1277 50  0000 C CNN
 F 2 "" H 5150 1450 50  0001 C CNN
@@
 $EndComp
 $Comp
-L Connector:USB_C_Plug_USB2.0 P?
+L Connector:USB_C_Plug_USB2.0 P1
 U 1 1 5E8910CA
 P 1600 4900
-F 0 "P?" H 1707 5767 50  0000 C CNN
+F 0 "P1" H 1707 5767 50  0000 C CNN
 F 1 "USB_C_Plug_USB2.0" H 1707 5676 50  0000 C CNN
-F 2 "" H 1750 4900 50  0001 C CNN
+F 2 "ASSETS:USB_C_Receptacle_HRO_TYPE-C-31-M-12" H 1750 4900 50  0001 C CNN
 F 3 "https://www.usb.org/sites/default/files/documents/usb_type-c.zip" H 1750 4900 50  0001 C CNN
 	1    1600 4900
@@
 	3150 4800 2750 4800
 $Comp
-L Power_Protection:SP0503BAHT D?
+L Power_Protection:SP0503BAHT D2
 U 1 1 5E8953CE
 P 2750 5400
-F 0 "D?" H 2955 5446 50  0000 L CNN
+F 0 "D2" H 2955 5446 50  0000 L CNN
 F 1 "SP0503BAHT" H 2955 5355 50  0000 L CNN
 F 2 "Package_TO_SOT_SMD:SOT-143" H 2975 5350 50  0001 L CNN
@@
 	2750 5600 2750 5800
 $Comp
-L power:GND #PWR?
+L power:GND #PWR0136
 U 1 1 5E89962A
 P 2750 5800
-F 0 "#PWR?" H 2750 5550 50  0001 C CNN
+F 0 "#PWR0136" H 2750 5550 50  0001 C CNN
 F 1 "GND" H 2755 5627 50  0000 C CNN
 F 2 "" H 2750 5800 50  0001 C CNN
@@
 	1600 6050 1600 5800
 $Comp
-L power:GND #PWR?
+L power:GND #PWR0137
 U 1 1 5E89B01C
 P 1450 6400
-F 0 "#PWR?" H 1450 6150 50  0001 C CNN
+F 0 "#PWR0137" H 1450 6150 50  0001 C CNN
 F 1 "GND" H 1455 6227 50  0000 C CNN
 F 2 "" H 1450 6400 50  0001 C CNN
@@
 	1450 6050 1600 6050
 $Comp
-L Device:R_Small R?
+L Device:R_Small R14
 U 1 1 5E89E449
 P 9050 4600
-F 0 "R?" H 9109 4646 50  0000 L CNN
+F 0 "R14" H 9109 4646 50  0000 L CNN
 F 1 "22.1K" H 9109 4555 50  0000 L CNN
-F 2 "" H 9050 4600 50  0001 C CNN
+F 2 "Resistor_SMD:R_0603_1608Metric" H 9050 4600 50  0001 C CNN
 F 3 "~" H 9050 4600 50  0001 C CNN
 	1    9050 4600
@@
 $EndComp
 $Comp
-L Device:R_Small R?
+L Device:R_Small R15
 U 1 1 5E89E78A
 P 9050 5050
-F 0 "R?" H 9109 5096 50  0000 L CNN
+F 0 "R15" H 9109 5096 50  0000 L CNN
 F 1 "47.5K" H 9109 5005 50  0000 L CNN
-F 2 "" H 9050 5050 50  0001 C CNN
+F 2 "Resistor_SMD:R_0603_1608Metric" H 9050 5050 50  0001 C CNN
 F 3 "~" H 9050 5050 50  0001 C CNN
 	1    9050 5050
@@
 	9050 5150 9050 5350
 $Comp
-L power:GND #PWR?
+L power:GND #PWR0138
 U 1 1 5E8A2860
 P 9050 5350
-F 0 "#PWR?" H 9050 5100 50  0001 C CNN
+F 0 "#PWR0138" H 9050 5100 50  0001 C CNN
 F 1 "GND" H 9055 5177 50  0000 C CNN
 F 2 "" H 9050 5350 50  0001 C CNN
@@
 NoConn ~ 4950 3600
 Text GLabel 6050 3700 2    50   Input ~ 0
-RXD
+PC4
 Text GLabel 6050 3800 2    50   Input ~ 0
-TXD
+PC5
 NoConn ~ 3750 3700
 Wire Wire Line
@@
 	3000 3800 3000 3900
 $Comp
-L Device:R_Small R?
+L Device:R_Small R10
 U 1 1 5E8B5C1A
 P 3000 4000
-F 0 "R?" H 3059 4046 50  0000 L CNN
+F 0 "R10" H 3059 4046 50  0000 L CNN
 F 1 "1K" H 3059 3955 50  0000 L CNN
-F 2 "" H 3000 4000 50  0001 C CNN
+F 2 "Resistor_SMD:R_0603_1608Metric" H 3000 4000 50  0001 C CNN
 F 3 "~" H 3000 4000 50  0001 C CNN
 	1    3000 4000
@@
 	3000 4100 3000 4150
 $Comp
-L power:GND #PWR?
+L power:GND #PWR0139
 U 1 1 5E8B78DA
 P 3000 4150
-F 0 "#PWR?" H 3000 3900 50  0001 C CNN
+F 0 "#PWR0139" H 3000 3900 50  0001 C CNN
 F 1 "GND" V 3005 4022 50  0000 R CNN
 F 2 "" H 3000 4150 50  0001 C CNN
@@
 	4400 5100 4450 5100
 $Comp
-L power:GND #PWR?
+L power:GND #PWR0140
 U 1 1 5E87A484
 P 4400 5250
-F 0 "#PWR?" H 4400 5000 50  0001 C CNN
+F 0 "#PWR0140" H 4400 5000 50  0001 C CNN
 F 1 "GND" H 4405 5077 50  0000 C CNN
 F 2 "" H 4400 5250 50  0001 C CNN
@@
 	4950 3800 5450 3800
 $Comp
-L Device:LED D?
+L Device:LED D3
 U 1 1 5E8819A9
 P 5450 3350
-F 0 "D?" V 5489 3233 50  0000 R CNN
+F 0 "D3" V 5489 3233 50  0000 R CNN
 F 1 "LED" V 5398 3233 50  0000 R CNN
-F 2 "" H 5450 3350 50  0001 C CNN
+F 2 "LED_SMD:LED_0805_2012Metric_Pad1.15x1.40mm_HandSolder" H 5450 3350 50  0001 C CNN
 F 3 "~" H 5450 3350 50  0001 C CNN
 	1    5450 3350
@@
 $EndComp
 $Comp
-L Device:LED D?
+L Device:LED D4
 U 1 1 5E8821FD
 P 5850 3350
-F 0 "D?" V 5889 3233 50  0000 R CNN
+F 0 "D4" V 5889 3233 50  0000 R CNN
 F 1 "LED" V 5798 3233 50  0000 R CNN
-F 2 "" H 5850 3350 50  0001 C CNN
+F 2 "LED_SMD:LED_0805_2012Metric_Pad1.15x1.40mm_HandSolder" H 5850 3350 50  0001 C CNN
 F 3 "~" H 5850 3350 50  0001 C CNN
 	1    5850 3350
@@
 	5450 3800 5850 3800
 $Comp
-L Device:R_Small R?
+L Device:R_Small R12
 U 1 1 5E88628E
 P 5450 2850
-F 0 "R?" H 5509 2896 50  0000 L CNN
+F 0 "R12" H 5509 2896 50  0000 L CNN
 F 1 "1K" H 5509 2805 50  0000 L CNN
-F 2 "" H 5450 2850 50  0001 C CNN
+F 2 "Resistor_SMD:R_0603_1608Metric" H 5450 2850 50  0001 C CNN
 F 3 "~" H 5450 2850 50  0001 C CNN
 	1    5450 2850
@@
 	5850 2500 5850 2750
 $Comp
-L Device:R_Small R?
+L Device:R_Small R13
 U 1 1 5E88ACF3
 P 5850 2850
-F 0 "R?" H 5909 2896 50  0000 L CNN
+F 0 "R13" H 5909 2896 50  0000 L CNN
 F 1 "1K" H 5909 2805 50  0000 L CNN
-F 2 "" H 5850 2850 50  0001 C CNN
+F 2 "Resistor_SMD:R_0603_1608Metric" H 5850 2850 50  0001 C CNN
 F 3 "~" H 5850 2850 50  0001 C CNN
 	1    5850 2850
@@
 	5650 2500 5850 2500
 Text GLabel 5650 2350 1    50   Input ~ 0
-+3.3v
++3.3V
 Wire Notes Line
 	7350 2000 7350 6100

Commit message: Add files via upload
Connections:
- net PC4: now also D4.1 (K)
- net PC5: no longer D4.1 (K)
- net D+: now reaches D2.4 (K), P1.A6 (D+), U3.3 (D+)
- net D-: now reaches D2.3 (K), P1.A7 (D-), U3.4 (D-)
Changed lines of the file:
@@
 P 3900 1050
 F 0 "C20" H 3700 1100 50  0000 L CNN
-F 1 "4.7U" H 3500 1000 50  0000 L CNN
+F 1 "4.7U" H 3700 950 50  0000 L CNN
 F 2 "Capacitor_SMD:C_0402_1005Metric" H 3900 1050 50  0001 C CNN
 F 3 "~" H 3900 1050 50  0001 C CNN
@@
 NoConn ~ 4950 4600
 Wire Wire Line
-	4950 3700 6050 3700
+	4950 3700 5850 3700
 Wire Wire Line
 	4950 3800 5450 3800
@@
 $EndComp
 Wire Wire Line
-	5850 3500 5850 3800
-Connection ~ 5850 3800
-Wire Wire Line
-	5850 3800 6050 3800
-Wire Wire Line
 	5450 3500 5450 3800
 Connection ~ 5450 3800
-Wire Wire Line
-	5450 3800 5850 3800
 $Comp
 L Device:R_Small R12
@@
 Wire Wire Line
 	2300 4300 2200 4300
+Wire Wire Line
+	5450 3800 6050 3800
+Wire Wire Line
+	5850 3500 5850 3700
+Connection ~ 5850 3700
+Wire Wire Line
+	5850 3700 6050 3700
+Text Label 3250 4400 0    50   ~ 0
+D+
+Text Label 3250 4500 0    50   ~ 0
+D-
 $EndSCHEMATC

Commit message: Add files via upload
Parts:
- removed R14: 22.1K, Resistor_SMD:R_0603_1608Metric, symbol Device:R_Small
- removed R15: 47.5K, Resistor_SMD:R_0603_1608Metric, symbol Device:R_Small
Changed lines of the file:
@@
 $Descr User 7874 7874
 encoding utf-8
-Sheet 5 7
+Sheet 5 6
 Title ""
 Date ""
@@
 Wire Wire Line
 	1450 6050 1600 6050
-$Comp
-L Device:R_Small R14
-U 1 1 5E89E449
-P 9050 4600
-F 0 "R14" H 9109 4646 50  0000 L CNN
-F 1 "22.1K" H 9109 4555 50  0000 L CNN
-F 2 "Resistor_SMD:R_0603_1608Metric" H 9050 4600 50  0001 C CNN
-F 3 "~" H 9050 4600 50  0001 C CNN
-	1    9050 4600
-	1    0    0    -1
-$EndComp
-$Comp
-L Device:R_Small R15
-U 1 1 5E89E78A
-P 9050 5050
-F 0 "R15" H 9109 5096 50  0000 L CNN
-F 1 "47.5K" H 9109 5005 50  0000 L CNN
-F 2 "Resistor_SMD:R_0603_1608Metric" H 9050 5050 50  0001 C CNN
-F 3 "~" H 9050 5050 50  0001 C CNN
-	1    9050 5050
-	1    0    0    -1
-$EndComp
-Wire Wire Line
-	9050 4950 9050 4850
-Wire Wire Line
-	9050 4500 9050 4300
-Text GLabel 9050 4300 1    50   Input ~ 0
-+5V
-Wire Wire Line
-	9050 5150 9050 5350
-$Comp
-L power:GND #PWR0138
-U 1 1 5E8A2860
-P 9050 5350
-F 0 "#PWR0138" H 9050 5100 50  0001 C CNN
-F 1 "GND" H 9055 5177 50  0000 C CNN
-F 2 "" H 9050 5350 50  0001 C CNN
-F 3 "" H 9050 5350 50  0001 C CNN
-	1    9050 5350
-	1    0    0    -1
-$EndComp
-Wire Wire Line
-	9050 4850 9400 4850
-Connection ~ 9050 4850
-Wire Wire Line
-	9050 4850 9050 4700
-Text Label 9400 4850 0    50   ~ 0
-IO
 NoConn ~ 4950 4300
 NoConn ~ 4950 4400
