File: STM32G473RET6 Development Board/_autosave-Dev_Pro.kicad_pcb (KiCad board)
At the start: 2 copper layers, 40 x 90 mm, 61 parts, among them IC1 STM32G473RET6, J1 Screw_Terminal_01x02, J2 USB_C_Receptacle_USB2.0, J3 Conn_01x25, J6 Conn_01x25, P1 USB_C_Plug_USB2.0, U1 AP2127R-3.3, U3 CP2102N-A01-GQFN24, U6 IRF7205TRPB

Commit message: Add files via upload
Parts:
- added ?: , , F.Cu at (148.5, 139.2)
Changed lines of the file:
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@@
   (general
     (thickness 1.6)
-    (drawings 78)
+    (drawings 76)
     (tracks 824)
     (zones 0)
-    (modules 61)
+    (modules 62)
     (nets 92)
   )
   (page A4)
   (layers
-    (0 F.Cu signal hide)
-    (31 B.Cu signal hide)
-    (32 B.Adhes user hide)
-    (33 F.Adhes user hide)
-    (34 B.Paste user hide)
-    (35 F.Paste user hide)
-    (36 B.SilkS user hide)
-    (37 F.SilkS user hide)
-    (38 B.Mask user hide)
-    (39 F.Mask user hide)
-    (40 Dwgs.User user hide)
-    (41 Cmts.User user hide)
-    (42 Eco1.User user hide)
-    (43 Eco2.User user hide)
+    (0 F.Cu signal)
+    (31 B.Cu signal)
+    (32 B.Adhes user)
+    (33 F.Adhes user)
+    (34 B.Paste user)
+    (35 F.Paste user)
+    (36 B.SilkS user)
+    (37 F.SilkS user)
+    (38 B.Mask user)
+    (39 F.Mask user)
+    (40 Dwgs.User user)
+    (41 Cmts.User user)
+    (42 Eco1.User user)
+    (43 Eco2.User user)
     (44 Edge.Cuts user)
-    (45 Margin user hide)
-    (46 B.CrtYd user hide)
-    (47 F.CrtYd user hide)
-    (48 B.Fab user hide)
-    (49 F.Fab user hide)
+    (45 Margin user)
+    (46 B.CrtYd user)
+    (47 F.CrtYd user)
+    (48 B.Fab user)
+    (49 F.Fab user)
   )
   (setup
@@
       (outputformat 1)
       (mirror false)
-      (drillshape 1)
+      (drillshape 0)
       (scaleselection 1)
-      (outputdirectory ""))
+      (outputdirectory "GERBER/"))
   )
   (net 0 "")
@@
     (uvia_drill 0.1)
   )
+  (module "" (layer F.Cu)
+    (at 148.5 139.25)
+    (fp_text reference "" (at 134.25 81.1875) (layer F.SilkS)
+      (effects (font (size 1.27 1.27) (thickness 0.15)))
+    )
+    (fp_text value "" (at 134.25 81.1875) (layer F.SilkS)
+      (effects (font (size 1.27 1.27) (thickness 0.15)))
+    )
+    (fp_text user "USB to UART" (at 0.25 0.75) (layer F.SilkS)
+      (effects (font (size 1 1) (thickness 0.15)))
+    )
+  )
   (module Resistor_SMD:R_0603_1608Metric (layer B.Cu)
     (at 134.25 81.1875 270)
@@
       (effects (font (size 1 1) (thickness 0.15)) (justify mirror))
     )
-    (fp_text value Conn_01x25 (at 0 -63.29) (layer B.Fab)
+    (fp_text value Conn_01x25 (at 4.25 -63.77) (layer B.Fab)
       (effects (font (size 1 1) (thickness 0.15)) (justify mirror))
     )
@@
       (effects (font (size 1 1) (thickness 0.15)) (justify mirror))
     )
-    (fp_text value Conn_01x25 (at 0 -63.29) (layer B.Fab)
+    (fp_text value Conn_01x25 (at -7.25 -54.27) (layer B.Fab)
       (effects (font (size 1 1) (thickness 0.15)) (justify mirror))
     )
@@
       (effects (font (size 1 1) (thickness 0.15)))
     )
-    (fp_text value USB_C_Receptacle_USB2.0 (at 0 5.1) (layer F.Fab)
+    (fp_text value USB_C_Receptacle_USB2.0 (at -0.75 -0.75) (layer F.Fab)
       (effects (font (size 1 1) (thickness 0.15)))
     )
@@
       (effects (font (size 1 1) (thickness 0.15)))
     )
-    (fp_text value USB_C_Plug_USB2.0 (at 0 5.1) (layer F.Fab)
+    (fp_text value USB_C_Plug_USB2.0 (at -0.25 -1) (layer F.Fab)
       (effects (font (size 1 1) (thickness 0.15)))
     )
@@
       (effects (font (size 1 1) (thickness 0.15)))
     )
-    (fp_text value Conn_ARM_JTAG_SWD_10 (at 0 4.235) (layer F.Fab)
+    (fp_text value Conn_ARM_JTAG_SWD_10 (at 5 1.25) (layer F.Fab)
       (effects (font (size 1 1) (thickness 0.15)))
     )
@@
       (effects (font (size 1 1) (thickness 0.15)))
     )
-    (fp_text value Conn_01x04 (at 3 7.45) (layer F.Fab)
+    (fp_text value Conn_01x04 (at 2.25 3) (layer F.Fab)
       (effects (font (size 1 1) (thickness 0.15)))
     )
@@
       (effects (font (size 1 1) (thickness 0.15)))
     )
-    (fp_text value Conn_01x04 (at 3 7.45) (layer F.Fab)
+    (fp_text value Conn_01x04 (at 3 2.75) (layer F.Fab)
       (effects (font (size 1 1) (thickness 0.15)))
     )
@@
     (descr "JST EH series connector, S2B-EH (http://www.jst-mfg.com/product/pdf/eng/eEH.pdf), generated with kicad-footprint-generator")
     (tags "connector JST EH horizontal")
-    (fp_text reference J1 (at 1.25 -7.9) (layer F.SilkS)
-      (effects (font (size 1 1) (thickness 0.15)))
-    )
-    (fp_text value Screw_Terminal_01x02 (at 1.25 2.7) (layer F.Fab)
+    (fp_text reference J1 (at 1.5 3) (layer F.SilkS)
+      (effects (font (size 1 1) (thickness 0.15)))
+    )
+    (fp_text value Screw_Terminal_01x02 (at 6 3) (layer F.Fab)
       (effects (font (size 1 1) (thickness 0.15)))
     )
@@
   (gr_line (start 146.5 61.25) (end 150.5 61.25) (layer Edge.Cuts) (width 0.05))
   (gr_line (start 168.5 108.5) (end 168.5 104.5) (layer Edge.Cuts) (width 0.05))
-  (gr_arc (start 171.25 104.75) (end 170.25 104.75) (angle -180) (layer F.SilkS) (width 0.12))
-  (gr_arc (start 171.25 108.75) (end 172.25 108.75) (angle -180) (layer F.SilkS) (width 0.12))
   (gr_line (start 148.5 61.25) (end 148.5 106.25) (layer Dwgs.User) (width 0.15))
   (gr_line (start 148.5 107.25) (end 148.5 155.25) (layer Dwgs.User) (width 0.15))
