File: Handheld GPS Tracker/Tracker.sch (KiCad schematic (older format))
At the start: 0 parts

Commit message: Add files via upload
Changed lines of the file:
@@
 $Descr User 7874 8662
 encoding utf-8
-Sheet 1 7
+Sheet 1 6
 Title ""
 Date ""
@@
 $EndSheet
 $Sheet
-S 700  3100 3000 1600
-U 5E919742
-F0 "FLASH" 50
-F1 "FLASH.sch" 50
-$EndSheet
-$Sheet
-S 4100 3100 3000 1600
+S 700  3050 3000 1600
 U 5E919744
 F0 "GNSS" 50
@@
 $EndSheet
 $Sheet
-S 700  5000 3000 1600
+S 4100 3050 3000 1600
 U 5E919796
 F0 "DISPLAY" 50
@@
 $EndSheet
 $Sheet
-S 4100 5000 3000 1600
+S 2400 5050 3000 1600
 U 5E919798
 F0 "BATTERY" 50
