File: Handheld GPS Tracker/BATTERY.sch (KiCad schematic (older format))
At the start: 0 parts

Commit message: Add files via upload
Parts:
- added C?: 4.7U, symbol Device:C_Small
- added D? (x2): LED, symbol Device:LED
- added J?: Conn_01x02, symbol Connector_Generic:Conn_01x02
- added P?: USB_C_Plug_USB2.0, symbol Connector:USB_C_Plug_USB2.0
- added R? (x2): R_Small, symbol Device:R_Small
- added R?: 46.4K, symbol Device:R_Small
- added R?: 1.18K, symbol Device:R_Small
- added R?: 1.13, symbol Device:R_Small
- added U?: BQ24072RGT, Package_DFN_QFN:VQFN-16-1EP_3x3mm_P0.5mm_EP1.6x1.6mm, symbol Battery_Management:BQ24072RGT
Connections:
- new net: D?.2 (A), R?.2 (x2)
- new net +3V3: R?.1, R?.1, U?.6 (EN1)
- new net BAT: U?.2 (BAT), U?.3 (BAT)
- new net BATTERY: C?.2, J?.2 (Pin_2)
- new net CE: U?.4 (~CE)
- new net CHG: D?.1 (K), U?.9 (~CHG)
- new net D+: P?.A6 (D+)
- new net D-: P?.A7 (D-)
- new net GND: C?.1, J?.1 (Pin_1), P?.A1 (GND), P?.A12 (GND), P?.B1 (GND), P?.B12 (GND), P?.S1 (SHIELD), R?.1, R?.1, R?.1, U?.17 (VSS), U?.5 (EN2), U?.8 (VSS)
- new net ILIM: U?.12 (ILIM)
- new net ILM: R?.2
- new net IN: U?.13 (IN)
- new net ISET: R?.2, U?.16 (ISET)
- new net OUT: U?.10 (OUT), U?.11 (OUT)
- new net PGOOD: D?.1 (K), U?.7 (~PGOOD)
- new net TD: U?.15 (TD)
- new net TMR: R?.2, U?.14 (TMR)
- new net TS: U?.1 (TS)
- new net VBUS: P?.A4 (VBUS), P?.A9 (VBUS), P?.B4 (VBUS), P?.B9 (VBUS)
- no-connect marks 0 -> 2

Commit message: Add files via upload
Parts:
- added C37: C_Small, symbol Device:C_Small
- added C39: 0.47U, symbol Device:C_Small
- added R14: R_Small, symbol Device:R_Small
- added R15: 10K, symbol Device:R_Small
- added SW1: SW_SPDT, symbol Switch:SW_SPDT
- added U10: BQ27441-G1, Package_SON:Texas_S-PDSO-N12, symbol Battery_Management:BQ27441-G1
- added U8: LT1129-3.3_SO8, Package_SO:SOIC-8_3.9x4.9mm_P1.27mm, symbol Regulator_Linear:LT1129-3.3_SO8
- gave numbers to parts that had none: 11
Connections:
- net BAT is gone; now on net BATTERY: U9.2 (BAT), U9.3 (BAT)
- net ILM is gone; now on net ILIM: R11.2
- net IN is gone; now on net VBUS: U9.13 (IN)
- net TD is gone; now on net GND: U9.15 (TD)
- net +3V3: now also C37.1, U8.1 (OUT), U8.2 (SENSE)
- net BATTERY: now also R14.2, SW1.1 (A), U10.6 (BAT), U10.8 (SRP)
- net CE: now also SW1.2 (B), U8.5 (~SHDN)
- net GND: now also C37.2, C39.1, R15.2, SW1.3 (C), U10.13 (PAD), U10.3 (VSS), U8.3 (GND), U8.6 (GND), U8.7 (GND)
- net D+: no longer names the net of P1.A6 (D+)
- net D-: no longer names the net of P1.A7 (D-)
- net OUT renamed VDD
- net VDD: now also R14.1, U10.7 (SRN), U8.8 (IN)
- net TS: no longer names the net of U9.1 (TS)
- new net: R15.1, U10.10 (BIN)
- new net: C39.2, U10.5 (VDD)
- new net GPOUT: U10.12 (GPOUT)
- new net SCL: U10.2 (SCL)
- new net SDA: U10.1 (SDA)
- no-connect marks 2 -> 5
Other:
- note added: "BAT PROT &\nCHARGING"
- note added: "FUEL\nGAUGE"
- note added: "USB"

Commit message: Add files via upload
Parts:
- C37, C38, C39: footprint (none) -> Capacitor_SMD:C_0603_1608Metric
- D1, D2: footprint (none) -> Diode_SMD:D_0603_1608Metric
- P1: footprint (none) -> ASSETS:USB_C_Receptacle_HRO_TYPE-C-31-M-12
- R10, R11, R12, R13, R14, R15, R9: footprint (none) -> Resistor_SMD:R_0402_1005Metric
- SW1: footprint (none) -> Button_Switch_SMD:SW_SPDT_PCM12
Changed lines of the file:
@@
 F 0 "D2" H 1743 5266 50  0000 C CNN
 F 1 "LED" H 1743 5175 50  0000 C CNN
-F 2 "" H 1750 5050 50  0001 C CNN
+F 2 "Diode_SMD:D_0603_1608Metric" H 1750 5050 50  0001 C CNN
 F 3 "~" H 1750 5050 50  0001 C CNN
 	1    1750 5050
@@
 F 0 "R13" V 1954 5050 50  0000 C CNN
 F 1 "R_Small" V 2045 5050 50  0000 C CNN
-F 2 "" H 2150 5050 50  0001 C CNN
+F 2 "Resistor_SMD:R_0402_1005Metric" H 2150 5050 50  0001 C CNN
 F 3 "~" H 2150 5050 50  0001 C CNN
 	1    2150 5050
@@
 F 0 "P1" H 1607 2517 50  0000 C CNN
 F 1 "USB_C_Plug_USB2.0" H 1607 2426 50  0000 C CNN
-F 2 "" H 1650 1650 50  0001 C CNN
+F 2 "ASSETS:USB_C_Receptacle_HRO_TYPE-C-31-M-12" H 1650 1650 50  0001 C CNN
 F 3 "https://www.usb.org/sites/default/files/documents/usb_type-c.zip" H 1650 1650 50  0001 C CNN
 	1    1500 1650
@@
 F 0 "C38" H 4458 3954 50  0000 R CNN
 F 1 "4.7U" H 4458 4045 50  0000 R CNN
-F 2 "" H 4550 4000 50  0001 C CNN
+F 2 "Capacitor_SMD:C_0603_1608Metric" H 4550 4000 50  0001 C CNN
 F 3 "~" H 4550 4000 50  0001 C CNN
 	1    4550 4000
@@
 F 0 "R9" V 1629 3500 50  0000 C CNN
 F 1 "46.4K" V 1720 3500 50  0000 C CNN
-F 2 "" H 1825 3500 50  0001 C CNN
+F 2 "Resistor_SMD:R_0402_1005Metric" H 1825 3500 50  0001 C CNN
 F 3 "~" H 1825 3500 50  0001 C CNN
 	1    1825 3500
@@
 F 0 "R11" V 1629 4325 50  0000 C CNN
 F 1 "1.18K" V 1720 4325 50  0000 C CNN
-F 2 "" H 1825 4325 50  0001 C CNN
+F 2 "Resistor_SMD:R_0402_1005Metric" H 1825 4325 50  0001 C CNN
 F 3 "~" H 1825 4325 50  0001 C CNN
 	1    1825 4325
@@
 F 0 "R10" V 1629 3925 50  0000 C CNN
 F 1 "1.13" V 1720 3925 50  0000 C CNN
-F 2 "" H 1825 3925 50  0001 C CNN
+F 2 "Resistor_SMD:R_0402_1005Metric" H 1825 3925 50  0001 C CNN
 F 3 "~" H 1825 3925 50  0001 C CNN
 	1    1825 3925
@@
 F 0 "D1" H 1718 5741 50  0000 C CNN
 F 1 "LED" H 1718 5650 50  0000 C CNN
-F 2 "" H 1725 5525 50  0001 C CNN
+F 2 "Diode_SMD:D_0603_1608Metric" H 1725 5525 50  0001 C CNN
 F 3 "~" H 1725 5525 50  0001 C CNN
 	1    1725 5525
@@
 F 0 "R12" V 1929 5525 50  0000 C CNN
 F 1 "R_Small" V 2020 5525 50  0000 C CNN
-F 2 "" H 2125 5525 50  0001 C CNN
+F 2 "Resistor_SMD:R_0402_1005Metric" H 2125 5525 50  0001 C CNN
 F 3 "~" H 2125 5525 50  0001 C CNN
 	1    2125 5525
@@
 F 0 "C39" V 6546 5225 50  0000 C CNN
 F 1 "0.47U" V 6637 5225 50  0000 C CNN
-F 2 "" H 6775 5225 50  0001 C CNN
+F 2 "Capacitor_SMD:C_0603_1608Metric" H 6775 5225 50  0001 C CNN
 F 3 "~" H 6775 5225 50  0001 C CNN
 	1    6775 5225
@@
 F 0 "R14" H 4284 5871 50  0000 L CNN
 F 1 "R_Small" H 4284 5780 50  0000 L CNN
-F 2 "" H 4225 5825 50  0001 C CNN
+F 2 "Resistor_SMD:R_0402_1005Metric" H 4225 5825 50  0001 C CNN
 F 3 "~" H 4225 5825 50  0001 C CNN
 	1    4225 5825
@@
 F 0 "R15" H 5059 6246 50  0000 L CNN
 F 1 "10K" H 5059 6155 50  0000 L CNN
-F 2 "" H 5000 6200 50  0001 C CNN
+F 2 "Resistor_SMD:R_0402_1005Metric" H 5000 6200 50  0001 C CNN
 F 3 "~" H 5000 6200 50  0001 C CNN
 	1    5000 6200
@@
 F 0 "C37" H 2767 6571 50  0000 L CNN
 F 1 "C_Small" H 2767 6480 50  0000 L CNN
-F 2 "" H 2675 6525 50  0001 C CNN
+F 2 "Capacitor_SMD:C_0603_1608Metric" H 2675 6525 50  0001 C CNN
 F 3 "~" H 2675 6525 50  0001 C CNN
 	1    2675 6525
@@
 F 0 "SW1" H 1775 7860 50  0000 C CNN
 F 1 "SW_SPDT" H 1775 7769 50  0000 C CNN
-F 2 "" H 1775 7575 50  0001 C CNN
+F 2 "Button_Switch_SMD:SW_SPDT_PCM12" H 1775 7575 50  0001 C CNN
 F 3 "~" H 1775 7575 50  0001 C CNN
 	1    1775 7575
