File: Handheld GPS Tracker/IMU.sch (KiCad schematic (older format))
At the start: 11 parts

Commit message: Add files via upload
Parts:
- gave numbers to parts that had none: 11
Connections:
- net at U3.27 (XIN32): now also C24.2, Y2.2
Changed lines of the file:
@@
 $Descr User 7874 8661
 encoding utf-8
-Sheet 3 7
+Sheet 3 6
 Title ""
 Date ""
@@
 $EndDescr
 $Comp
-L Sensor_Motion:BNO055 U?
+L Sensor_Motion:BNO055 U3
 U 1 1 5E99CAD9
 P 3950 3775
-F 0 "U?" H 4325 4500 50  0000 C CNN
+F 0 "U3" H 4325 4500 50  0000 C CNN
 F 1 "BNO055" H 4325 4425 50  0000 C CNN
 F 2 "Package_LGA:LGA-28_5.2x3.8mm_P0.5mm" H 4200 3125 50  0001 L CNN
@@
 	3050 4275 3050 4350
 $Comp
-L power:GNDD #PWR?
+L power:GNDD #PWR026
 U 1 1 5E99D698
 P 3050 4350
-F 0 "#PWR?" H 3050 4100 50  0001 C CNN
+F 0 "#PWR026" H 3050 4100 50  0001 C CNN
 F 1 "GNDD" H 3054 4195 50  0000 C CNN
 F 2 "" H 3050 4350 50  0001 C CNN
@@
 $EndComp
 $Comp
-L Device:Crystal_Small Y?
+L Device:Crystal_Small Y2
 U 1 1 5E99E50A
 P 5075 3500
-F 0 "Y?" V 5029 3588 50  0000 L CNN
+F 0 "Y2" V 5029 3588 50  0000 L CNN
 F 1 "32.768KHz" V 5120 3588 50  0000 L CNN
 F 2 "" H 5075 3500 50  0001 C CNN
@@
 	5075 3275 4550 3275
 Wire Wire Line
-	4575 3775 5075 3775
-Wire Wire Line
 	5075 3775 5075 3600
 $Comp
-L Device:C_Small C?
+L Device:C_Small C25
 U 1 1 5E99EDF3
 P 5800 3275
-F 0 "C?" V 5571 3275 50  0000 C CNN
+F 0 "C25" V 5571 3275 50  0000 C CNN
 F 1 "22P" V 5662 3275 50  0000 C CNN
 F 2 "" H 5800 3275 50  0001 C CNN
@@
 Connection ~ 5075 3275
 $Comp
-L Device:C_Small C?
+L Device:C_Small C24
 U 1 1 5E99F991
 P 5775 3775
-F 0 "C?" V 5546 3775 50  0000 C CNN
+F 0 "C24" V 5546 3775 50  0000 C CNN
 F 1 "22P" V 5637 3775 50  0000 C CNN
 F 2 "" H 5775 3775 50  0001 C CNN
@@
 	6150 3500 6150 3775
 $Comp
-L power:GND #PWR?
+L power:GND #PWR034
 U 1 1 5E9A0640
 P 6400 3575
-F 0 "#PWR?" H 6400 3325 50  0001 C CNN
+F 0 "#PWR034" H 6400 3325 50  0001 C CNN
 F 1 "GND" H 6405 3402 50  0000 C CNN
 F 2 "" H 6400 3575 50  0001 C CNN
@@
 $EndComp
 $Comp
-L Device:R_Small R?
+L Device:R_Small R4
 U 1 1 5E9A1F57
 P 2025 3625
-F 0 "R?" H 2084 3671 50  0000 L CNN
+F 0 "R4" H 2084 3671 50  0000 L CNN
 F 1 "4.7K" H 2084 3580 50  0000 L CNN
 F 2 "" H 2025 3625 50  0001 C CNN
@@
 $EndComp
 $Comp
-L Device:R_Small R?
+L Device:R_Small R6
 U 1 1 5E9A1FB2
 P 2775 3400
-F 0 "R?" H 2834 3446 50  0000 L CNN
+F 0 "R6" H 2834 3446 50  0000 L CNN
 F 1 "10K" H 2834 3355 50  0000 L CNN
 F 2 "" H 2775 3400 50  0001 C CNN
@@
 $EndComp
 $Comp
-L Device:R_Small R?
+L Device:R_Small R7
 U 1 1 5E9A20D5
 P 3275 2875
-F 0 "R?" H 3334 2921 50  0000 L CNN
+F 0 "R7" H 3334 2921 50  0000 L CNN
 F 1 "R_Small" H 3334 2830 50  0000 L CNN
 F 2 "" H 3275 2875 50  0001 C CNN
@@
 $EndComp
 $Comp
-L Device:R_Small R?
+L Device:R_Small R5
 U 1 1 5E9A21C5
 P 2425 3625
-F 0 "R?" H 2484 3671 50  0000 L CNN
+F 0 "R5" H 2484 3671 50  0000 L CNN
 F 1 "4.7K" H 2484 3580 50  0000 L CNN
 F 2 "" H 2425 3625 50  0001 C CNN
@@
 	2200 3375 2425 3375
 $Comp
-L power:+3.3V #PWR?
+L power:+3.3V #PWR023
 U 1 1 5E9A4B42
 P 2200 3250
-F 0 "#PWR?" H 2200 3100 50  0001 C CNN
+F 0 "#PWR023" H 2200 3100 50  0001 C CNN
 F 1 "+3.3V" H 2215 3423 50  0000 C CNN
 F 2 "" H 2200 3250 50  0001 C CNN
@@
 	2775 3300 2775 3075
 $Comp
-L power:+3.3V #PWR?
+L power:+3.3V #PWR024
 U 1 1 5E9A60EF
 P 2775 3075
-F 0 "#PWR?" H 2775 2925 50  0001 C CNN
+F 0 "#PWR024" H 2775 2925 50  0001 C CNN
 F 1 "+3.3V" H 2790 3248 50  0000 C CNN
 F 2 "" H 2775 3075 50  0001 C CNN
@@
 	3050 3775 3050 3800
 $Comp
-L power:GNDD #PWR?
+L power:GNDD #PWR025
 U 1 1 5E9A6FB9
 P 3050 3800
-F 0 "#PWR?" H 3050 3550 50  0001 C CNN
+F 0 "#PWR025" H 3050 3550 50  0001 C CNN
 F 1 "GNDD" V 3054 3690 50  0000 R CNN
 F 2 "" H 3050 3800 50  0001 C CNN
@@
 	3275 2775 3275 2650
 $Comp
-L power:+3.3V #PWR?
+L power:+3.3V #PWR027
 U 1 1 5E9A8A0B
 P 3275 2650
-F 0 "#PWR?" H 3275 2500 50  0001 C CNN
+F 0 "#PWR027" H 3275 2500 50  0001 C CNN
 F 1 "+3.3V" H 3290 2823 50  0000 C CNN
 F 2 "" H 3275 2650 50  0001 C CNN
@@
 RESET
 $Comp
-L power:+3.3V #PWR?
+L power:+3.3V #PWR031
 U 1 1 5E9AF414
 P 4050 2500
-F 0 "#PWR?" H 4050 2350 50  0001 C CNN
+F 0 "#PWR031" H 4050 2350 50  0001 C CNN
 F 1 "+3.3V" H 4065 2673 50  0000 C CNN
 F 2 "" H 4050 2500 50  0001 C CNN
@@
 $EndComp
 $Comp
-L Device:C_Small C?
+L Device:C_Small C22
 U 1 1 5E9AF6C1
 P 4350 2725
-F 0 "C?" H 4442 2771 50  0000 L CNN
+F 0 "C22" H 4442 2771 50  0000 L CNN
 F 1 "6.8N" H 4442 2680 50  0000 L CNN
 F 2 "" H 4350 2725 50  0001 C CNN
@@
 $EndComp
 $Comp
-L Device:C_Small C?
+L Device:C_Small C23
 U 1 1 5E9AFD3C
 P 4750 2725
-F 0 "C?" H 4842 2771 50  0000 L CNN
+F 0 "C23" H 4842 2771 50  0000 L CNN
 F 1 "120N" H 4842 2680 50  0000 L CNN
 F 2 "" H 4750 2725 50  0001 C CNN
@@
 	4550 2875 4750 2875
 $Comp
-L power:GNDD #PWR?
+L power:GNDD #PWR032
 U 1 1 5E9B3CEC
 P 4550 2925
-F 0 "#PWR?" H 4550 2675 50  0001 C CNN
+F 0 "#PWR032" H 4550 2675 50  0001 C CNN
 F 1 "GNDD" H 4554 2770 50  0000 C CNN
 F 2 "" H 4550 2925 50  0001 C CNN
@@
 	3850 2600 3850 2675
 $Comp
-L power:+3.3V #PWR?
+L power:+3.3V #PWR029
 U 1 1 5E9B4F88
 P 3850 2600
-F 0 "#PWR?" H 3850 2450 50  0001 C CNN
+F 0 "#PWR029" H 3850 2450 50  0001 C CNN
 F 1 "+3.3V" H 3865 2773 50  0000 C CNN
 F 2 "" H 3850 2600 50  0001 C CNN
@@
 $EndComp
 $Comp
-L Device:C_Small C?
+L Device:C_Small C21
 U 1 1 5E9B5288
 P 3575 2175
-F 0 "C?" H 3667 2221 50  0000 L CNN
+F 0 "C21" H 3667 2221 50  0000 L CNN
 F 1 "6.8N" H 3667 2130 50  0000 L CNN
 F 2 "" H 3575 2175 50  0001 C CNN
@@
 	3350 1975 3350 2050
 $Comp
-L power:GNDD #PWR?
+L power:GNDD #PWR028
 U 1 1 5E9B7CBE
 P 3350 2050
-F 0 "#PWR?" H 3350 1800 50  0001 C CNN
+F 0 "#PWR028" H 3350 1800 50  0001 C CNN
 F 1 "GNDD" H 3354 1895 50  0000 C CNN
 F 2 "" H 3350 2050 50  0001 C CNN
@@
 	4900 4075 4900 4175
 $Comp
-L power:GNDD #PWR?
+L power:GNDD #PWR033
 U 1 1 5E9BA519
 P 4900 4350
-F 0 "#PWR?" H 4900 4100 50  0001 C CNN
+F 0 "#PWR033" H 4900 4100 50  0001 C CNN
 F 1 "GNDD" H 4904 4195 50  0000 C CNN
 F 2 "" H 4900 4350 50  0001 C CNN
@@
 	4050 4600 4050 4475
 $Comp
-L power:GNDD #PWR?
+L power:GNDD #PWR030
 U 1 1 5E9BF855
 P 3950 4725
-F 0 "#PWR?" H 3950 4475 50  0001 C CNN
+F 0 "#PWR030" H 3950 4475 50  0001 C CNN
 F 1 "GNDD" H 3954 4570 50  0000 C CNN
 F 2 "" H 3950 4725 50  0001 C CNN
@@
 Wire Wire Line
 	3950 4600 4050 4600
+Wire Wire Line
+	4550 3775 5075 3775
 $EndSCHEMATC

Commit message: Add files via upload
Parts:
- C21, C22, C23, C24, C25: footprint (none) -> Capacitor_SMD:C_0603_1608Metric
- R4, R5, R6, R7: footprint (none) -> Resistor_SMD:R_0402_1005Metric
- Y2: footprint (none) -> Crystal:Crystal_SMD_0603-2Pin_6.0x3.5mm
Changed lines of the file:
@@
 F 0 "Y2" V 5029 3588 50  0000 L CNN
 F 1 "32.768KHz" V 5120 3588 50  0000 L CNN
-F 2 "" H 5075 3500 50  0001 C CNN
+F 2 "Crystal:Crystal_SMD_0603-2Pin_6.0x3.5mm" H 5075 3500 50  0001 C CNN
 F 3 "~" H 5075 3500 50  0001 C CNN
 	1    5075 3500
@@
 F 0 "C25" V 5571 3275 50  0000 C CNN
 F 1 "22P" V 5662 3275 50  0000 C CNN
-F 2 "" H 5800 3275 50  0001 C CNN
+F 2 "Capacitor_SMD:C_0603_1608Metric" H 5800 3275 50  0001 C CNN
 F 3 "~" H 5800 3275 50  0001 C CNN
 	1    5800 3275
@@
 F 0 "C24" V 5546 3775 50  0000 C CNN
 F 1 "22P" V 5637 3775 50  0000 C CNN
-F 2 "" H 5775 3775 50  0001 C CNN
+F 2 "Capacitor_SMD:C_0603_1608Metric" H 5775 3775 50  0001 C CNN
 F 3 "~" H 5775 3775 50  0001 C CNN
 	1    5775 3775
@@
 F 0 "R4" H 2084 3671 50  0000 L CNN
 F 1 "4.7K" H 2084 3580 50  0000 L CNN
-F 2 "" H 2025 3625 50  0001 C CNN
+F 2 "Resistor_SMD:R_0402_1005Metric" H 2025 3625 50  0001 C CNN
 F 3 "~" H 2025 3625 50  0001 C CNN
 	1    2025 3625
@@
 F 0 "R6" H 2834 3446 50  0000 L CNN
 F 1 "10K" H 2834 3355 50  0000 L CNN
-F 2 "" H 2775 3400 50  0001 C CNN
+F 2 "Resistor_SMD:R_0402_1005Metric" H 2775 3400 50  0001 C CNN
 F 3 "~" H 2775 3400 50  0001 C CNN
 	1    2775 3400
@@
 F 0 "R7" H 3334 2921 50  0000 L CNN
 F 1 "R_Small" H 3334 2830 50  0000 L CNN
-F 2 "" H 3275 2875 50  0001 C CNN
+F 2 "Resistor_SMD:R_0402_1005Metric" H 3275 2875 50  0001 C CNN
 F 3 "~" H 3275 2875 50  0001 C CNN
 	1    3275 2875
@@
 F 0 "R5" H 2484 3671 50  0000 L CNN
 F 1 "4.7K" H 2484 3580 50  0000 L CNN
-F 2 "" H 2425 3625 50  0001 C CNN
+F 2 "Resistor_SMD:R_0402_1005Metric" H 2425 3625 50  0001 C CNN
 F 3 "~" H 2425 3625 50  0001 C CNN
 	1    2425 3625
@@
 F 0 "C22" H 4442 2771 50  0000 L CNN
 F 1 "6.8N" H 4442 2680 50  0000 L CNN
-F 2 "" H 4350 2725 50  0001 C CNN
+F 2 "Capacitor_SMD:C_0603_1608Metric" H 4350 2725 50  0001 C CNN
 F 3 "~" H 4350 2725 50  0001 C CNN
 	1    4350 2725
@@
 F 0 "C23" H 4842 2771 50  0000 L CNN
 F 1 "120N" H 4842 2680 50  0000 L CNN
-F 2 "" H 4750 2725 50  0001 C CNN
+F 2 "Capacitor_SMD:C_0603_1608Metric" H 4750 2725 50  0001 C CNN
 F 3 "~" H 4750 2725 50  0001 C CNN
 	1    4750 2725
@@
 F 0 "C21" H 3667 2221 50  0000 L CNN
 F 1 "6.8N" H 3667 2130 50  0000 L CNN
-F 2 "" H 3575 2175 50  0001 C CNN
+F 2 "Capacitor_SMD:C_0603_1608Metric" H 3575 2175 50  0001 C CNN
 F 3 "~" H 3575 2175 50  0001 C CNN
 	1    3575 2175
