File: Dooms Day Comm/DISPLAY&LORA.sch (KiCad schematic (older format))
At the start: 0 parts

Commit message: Add files via upload
Parts:
- added C? (x21): C_Small, symbol Device:C_Small
- added C? (x4): 100P, symbol Device:C_Small
- added IC?: SX1278IMLTRT, QFN65P600X600X100-29N-D, symbol SX1278IMLTRT:SX1278IMLTRT
- added J?: LoRa Antenna, symbol Connector_Generic:Conn_01x02
- added L? (x6): L_Small, symbol Device:L_Small
- added R? (x2): R_Small, symbol Device:R_Small
- added U?: SPI_DISPLAY_3.2_INCH, ASSETS:ILI9341 TFT DISPLAY SPI, symbol ILI9341_SPI_DISPLAY:SPI_DISPLAY_3.2_INCH
- added U?: PE4259, symbol PE4259:PE4259
- added Y?: 32 MHz, symbol Device:Crystal_GND23_Small
Connections:
- new net: R?.2, U?.10 (ANODE)
- new net: C?.1, IC?.2 (VR_ANA)
- new net: C?.1, IC?.4 (VR_DIG)
- new net: C?.1, C?.1, L?.1, L?.1
- new net: C?.2, L?.2
- new net: C?.1, C?.1, L?.1, L?.2
- new net: C?.1, C?.2, L?.1, U?.1 (RF1)
- new net: C?.2, J?.1 (Pin_1), L?.1
- new net: C?.2, U?.3 (RF2)
- new net: C?.1, U?.5 (RFC)
- new net: C?.1, R?.2
- new net: C?.1, L?.1, R?.1
- new net: C?.2, C?.2, L?.2
- new net +3V3: C?.1, C?.1, C?.1, C?.1, C?.1, C?.1, C?.1, C?.1, IC?.14 (VBAT_DIG), IC?.24 (VBAT_RF), IC?.3 (VBAT_ANA), R?.1, U?.6 (VDD), U?.9 (VCC)
- new net CLK: IC?.16 (SCK), U?.3 (SCL)
- new net CS: U?.5 (CS)
- new net GND: C?.1, C?.1, C?.2, C?.2, C?.2, C?.2, C?.2, C?.2, C?.2, C?.2, C?.2, C?.2, C?.2, C?.2, C?.2, C?.2, C?.2, C?.2, C?.2, C?.2, C?.2, IC?.15 (GND_1), IC?.21 (GND_2), IC?.22 (GND_3), IC?.23 (GND_4), IC?.26 (GND_5), J?.2 (Pin_2), U?.1 (GND), U?.11 (K1), U?.12 (K2), U?.13 (K3), U?.14 (K4), U?.2 (GND), U?.8 (GND), Y?.2, Y?.3
- new net MISO: IC?.17 (MISO), U?.6 (SDA)
- new net MOSI: IC?.18 (MOSI), U?.7 (SDO)
- new net NSS: IC?.19 (NSS)
- new net PA_BOOST: IC?.27 (PA_BOOST), L?.2
- new net RESET: IC?.7 (NRESET), U?.2 (RESET)
- new net RFI_LF: C?.1, IC?.1 (RFI_LF), L?.2
- new net RS: U?.4 (RS/A0)
- new net RXTX: IC?.20 (RXTX/RFMOD), U?.4 (CNTRL)
- new net VR_PA: C?.1, C?.1, IC?.25 (VR_PA), L?.2
- new net X+: U?.17 (X+)
- new net X-: U?.15 (X-), U?.18 (Y+)
- new net XTA: C?.1, IC?.5 (XTA), Y?.4
- new net XTB: C?.1, IC?.6 (XTB), Y?.1
- new net Y-: U?.16 (Y-)
- no-connect marks 0 -> 7
