File: Dooms Day Comm/FLASH&CAPTOUCH.sch (KiCad schematic (older format))
At the start: 7 parts

Commit message: Add files via upload
Parts:
- added J?: SLIDER, ASSETS:TOUCH_SLIDER, symbol Connector_Generic:Conn_01x08
- added J?: BUTTON 4, symbol Connector_Generic:Conn_01x01
- added J?: BUTTON 3, symbol Connector_Generic:Conn_01x01
- added J?: BUTTON 2, symbol Connector_Generic:Conn_01x01
- added J?: BUTTON 1, symbol Connector_Generic:Conn_01x01
- U?: symbol MPR121:MPR121 -> Trax-rescue:MPR121-MPR121
Connections:
- net at U?.10 (ELE2): now also J?.1 (Pin_1)
- net at U?.11 (ELE3): now also J?.1 (Pin_1)
- net at U?.12 (ELE4): now also J?.1 (Pin_1)
- net at U?.13 (ELE5): now also J?.2 (Pin_2)
- net at U?.14 (ELE6): now also J?.3 (Pin_3)
- net at U?.15 (ELE7): now also J?.4 (Pin_4)
- net at U?.16 (ELE8): now also J?.5 (Pin_5)
- net at U?.17 (ELE9): now also J?.6 (Pin_6)
- net at U?.18 (ELE10): now also J?.7 (Pin_7)
- net at U?.19 (ELE11): now also J?.8 (Pin_8)
- net at U?.8 (ELE0): now also J?.1 (Pin_1)
- net at U?.9 (ELE1): now also J?.1 (Pin_1)
Other:
- moved on the sheet: C?, R?, U?
