File: Dooms Day Comm/GNSS&POWER.sch (KiCad schematic (older format))
At the start: 28 parts

Commit message: Add files via upload
Parts:
- U?: symbol MCP73113_4:MCP73113_4 -> Trax-rescue:MCP73113_4-MCP73113_4
- U?: symbol Battery_MG:STC3117 -> Trax-rescue:STC3117-Battery_MG
Changed lines of the file:
@@
 $EndComp
 $Comp
-L MCP73113_4:MCP73113_4 U?
+L Trax-rescue:MCP73113_4-MCP73113_4 U?
 U 1 1 5E986C9A
 P 3580 5520
+AR Path="/5E986C9A" Ref="U?"  Part="1"
+AR Path="/5E97C7CB/5E986C9A" Ref="U?"  Part="1"
 F 0 "U?" H 3930 5685 50  0000 C CNN
 F 1 "MCP73113_4" H 3930 5594 50  0000 C CNN
@@
 SCL
 $Comp
-L Battery_MG:STC3117 U?
+L Trax-rescue:STC3117-Battery_MG U?
 U 1 1 5EA13B3B
 P 4650 6760
+AR Path="/5EA13B3B" Ref="U?"  Part="1"
+AR Path="/5E97C7CB/5EA13B3B" Ref="U?"  Part="1"
 F 0 "U?" H 5150 6825 50  0000 C CNN
 F 1 "STC3117" H 5150 6734 50  0000 C CNN
