File: GEOLOCX/DISPLAY&LORA.sch (KiCad schematic (older format))
At the start: 38 parts

Commit message: Add files via upload
Parts:
- IC2: renamed from IC?; footprint QFN65P600X600X100-29N-D -> ASSETS:QFN65P600X600X100-29N-D
- L1, L2, L3, L4, L5, L6: renamed from L?; footprint (none) -> Inductor_SMD:L_0402_1005Metric
- R2, R3: renamed from R?; footprint (none) -> Resistor_SMD:R_0603_1608Metric
- Y1: renamed from Y?; footprint (none) -> Crystal:Crystal_SMD_Abracon_ABM8G-4Pin_3.2x2.5mm
- gave numbers to parts that had none: 28
Connections:
- net CS renamed NSS_DISPLAY
- net NSS renamed NSS_LORA
- net RESET renamed LCD_RESET
- net LCD_RESET: no longer IC2.7 (NRESET)
- new net LORA_RESET: IC2.7 (NRESET)
