File: GEOLOCX/FLASH&CAPTOUCH.sch (KiCad schematic (older format))
At the start: 12 parts

Commit message: Add files via upload
Parts:
- R1: renamed from R?; footprint (none) -> Resistor_SMD:R_0603_1608Metric
- gave numbers to parts that had none: 11
Connections:
- no-connect marks 1 -> 2
