File: GEOLOCX/GNSS&POWER.sch (KiCad schematic (older format))
At the start: 28 parts

Commit message: Add files via upload
Parts:
- J8: renamed from J?; footprint (none) -> ASSETS:USB_C_Receptacle_HRO_TYPE-C-31-M-12
- L7: renamed from L?; footprint (none) -> Inductor_SMD:L_0402_1005Metric
- R4, R5, R6, R7, R8: renamed from R?; footprint (none) -> Resistor_SMD:R_0603_1608Metric
- U7: renamed from U?; footprint TESEO-LIV3F -> TESEO_LIV3R:TESEO-LIV3F
- U9: renamed from U?; footprint (none) -> ASSETS:B4327
- gave numbers to parts that had none: 19
