File: GEOLOCX/MCU.sch (KiCad schematic (older format))
At the start: 0 parts

Commit message: Add files via upload
Parts:
- added C30, C32, C34, C36, C38: 100N, symbol Device:C_Small
- added C31, C33, C35, C37, C39: 1U, symbol Device:C_Small
- added C40, C41: C_Small, symbol Device:C_Small
- added IC3: STM32G473RET6, QFP50P1200X1200X160-64N, symbol K_STM32G473RET6:STM32G473RET6
- added Y2: 32 MHz, Crystal:Crystal_SMD_Abracon_ABM8G-4Pin_3.2x2.5mm, symbol Device:Crystal_GND23_Small
Connections:
- new net +3V3: C30.2, C31.2, C32.2, C33.2, C34.2, C35.2, C36.2, C37.2, C38.2, C39.2, IC3.16 (VDD_1), IC3.28 (VREF+), IC3.29 (VDDA), IC3.32 (VDD_2), IC3.48 (VDD_3), IC3.64 (VDD_4)
- new net 1PPS: IC3.39 (PC7)
- new net ALM: IC3.44 (PA10)
- new net CD: IC3.43 (PA9)
- new net CLK: IC3.19 (PA5)
- new net D+: IC3.46 (PA12)
- new net D-: IC3.45 (PA11)
- new net GND: C30.1, C31.1, C32.1, C33.1, C34.1, C35.1, C36.1, C37.1, C38.1, C39.1, C40.2, C41.2, IC3.15 (VSS_1), IC3.27 (VSSA), IC3.31 (VSS_2), IC3.47 (VSS_3), IC3.63 (VSS_4), Y2.2, Y2.3
- new net IRQ: IC3.42 (PA8)
- new net LCD_RESET: IC3.26 (PB2)
- new net LORA_RESET: IC3.13 (PA1)
- new net MISO: IC3.20 (PA6)
- new net MOSI: IC3.21 (PA7)
- new net NRST: IC3.7 (PG10-NRST)
- new net NSS_DISPLAY: IC3.23 (PC5)
- new net NSS_FLASH: IC3.22 (PC4)
- new net NSS_LORA: IC3.24 (PB0)
- new net OSC8_IN: C40.1, IC3.5 (PF0-OSC_IN), Y2.1
- new net OSC8_OUT: C41.1, IC3.6 (PF1-OSC_OUT), Y2.4
- new net RS: IC3.25 (PB1)
- new net SCL: IC3.40 (PC8)
- new net SDA: IC3.41 (PC9)
- new net SWCLK: IC3.50 (PA14)
- new net SWDIO: IC3.49 (PA13)
- new net SYS_RSTN: IC3.37 (PB15)
- new net USART_RX: IC3.17 (PA3)
- new net USART_TX: IC3.14 (PA2)
- new net WAKE-UP: IC3.38 (PC6)
- new net X+: IC3.34 (PB12)
- new net X-: IC3.33 (PB11), IC3.36 (PB14)
- new net Y-: IC3.35 (PB13)
- no-connect marks 0 -> 22
