File: XESC v1/XESC.kicad_pcb (KiCad board)
At the start: 2 copper layers, 98 parts, among them IC1 STM32G473CEU6, J1 PHASE A, J2 PHASE A, J3 PHASE A, J4 PWR_IN, J5 GND, J6 UART, J7 SWD, Q1 QM6015D, U1 IR2101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

Commit message: Add files via upload
Parts:
- removed REF** (x2): MountingHole_2.2mm_M2_Pad_Via, MountingHole:MountingHole_2.2mm_M2_Pad_Via
- D3, R1, R10, R11, R6, R7, U3: moved to B.Cu
- moved D2 206.7 mm to (-26.0, 33.0)
- moved R3 189.2 mm to (-31.0, 38.0), turned to 90 degrees
- moved R2 180.4 mm to (6.00, 27.0), turned to 90 degrees
- moved R7 174.8 mm to (3.75, 12.0), turned to 270 degrees
- moved U2 174.5 mm to (-26.0, 37.0)
- moved R11 174.5 mm to (4.00, 24.0), turned to 270 degrees
- moved C2 171.3 mm to (-33.0, 29.0), turned to 180 degrees
- moved D3 170.5 mm to (12.1, 6.75), turned to 180 degrees
- moved L3 170.3 mm to (-33.0, 31.0), turned to 90 degrees
- moved C3 170.0 mm to (3.95, 5.25), turned to 180 degrees
- moved L1 168.1 mm to (4.00, 8.00), turned to 90 degrees
- moved C5 161.2 mm to (-26.0, 29.0), turned to 180 degrees
- moved C6 158.8 mm to (11.8, 5.25), turned to 0 degrees
- moved R6 158.2 mm to (20.0, 12.0), turned to 270 degrees
- moved U1 158.2 mm to (-26.0, 23.0)
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Connections:
- H1 pad 1: VDD -> Net-(H1-Pad1)
- H1 pad 2: Net-(H1-Pad2) -> VDD
- H2 pad 1: VDD -> Net-(H2-Pad1)
- H2 pad 2: Net-(H2-Pad2) -> VDD
- H2 pad 3: CONN_C -> CONN_B
- H3 pad 1: VDD -> Net-(H3-Pad1)
- H3 pad 2: Net-(H3-Pad2) -> VDD
- H3 pad 3: CONN_B -> CONN_C
- L1 pad 1: CONN_A -> Net-(L1-Pad1)
- L1 pad 2: Net-(L1-Pad2) -> CONN_A
- L2 pad 1: CONN_C -> Net-(L2-Pad1)
- L2 pad 2: Net-(L2-Pad2) -> CONN_B
- L3 pad 1: CONN_B -> Net-(L3-Pad1)
- L3 pad 2: Net-(L3-Pad2) -> CONN_C
- R10 pad 1: Net-(H3-Pad2) -> Net-(H2-Pad1)
- R11 pad 1: Net-(L3-Pad2) -> Net-(L2-Pad1)
- R6 pad 1: Net-(H1-Pad2) -> Net-(H1-Pad1)
- R7 pad 1: Net-(L1-Pad2) -> Net-(L1-Pad1)
- R8 pad 1: Net-(H2-Pad2) -> Net-(H3-Pad1)
- R9 pad 1: Net-(L2-Pad2) -> Net-(L3-Pad1)

Commit message: Add files via upload
Parts:
- removed C7, C8, C9: 4.7U, Capacitor_SMD:CP_Elec_4x3.9
- C1, C2, C3, C4, C5, C6: footprint Capacitor_SMD:CP_Elec_4x3.9 -> Capacitor_SMD:C_0805_2012Metric_Pad1.15x1.40mm_HandSolder
- C10, C11, C12, C13, C16, C17, C18, C19, C20, C21, C22: footprint Capacitor_SMD:C_0201_0603Metric -> Capacitor_SMD:C_0805_2012Metric_Pad1.15x1.40mm_HandSolder
- C14, C15: footprint Capacitor_SMD:C_0201_0603Metric -> Capacitor_SMD:C_0805_2012Metric_Pad1.15x1.40mm_HandSolder; moved to B.Cu
- C23, C24: footprint Capacitor_SMD:C_0201_0603Metric -> Capacitor_THT:CP_Radial_D25.0mm_P10.00mm_SnapIn
- D3, H1, H2, H3, U3: moved to F.Cu
- D4, D5, D6, D7, D8: footprint LED_SMD:LED_0201_0603Metric -> LED_SMD:LED_0805_2012Metric_Pad1.15x1.40mm_HandSolder
- J1, J2, J3, J4, J5: footprint ASSETS:PAD_5X5 -> ASSETS:PAD_7X6.75
- R1, R10, R6: footprint Resistor_SMD:R_0402_1005Metric -> Resistor_SMD:R_0805_2012Metric; moved to F.Cu
- R11, R12, R13, R14, R2, R24, R25, R26, R27, R28, R3, R4, R5, R7, R8: footprint Resistor_SMD:R_0402_1005Metric -> Resistor_SMD:R_0805_2012Metric
- R15, R16, R17, R18, R19, R20, R21, R22, R23, R9: footprint Resistor_SMD:R_0402_1005Metric -> Resistor_SMD:R_0805_2012Metric; moved to B.Cu
- moved R3 273.6 mm to (241.7, 15.5), turned to 0 degrees
- moved J2 244.6 mm to (236.3, 14.4)
- moved R2 210.0 mm to (214.8, 49.9), turned to 0 degrees
- moved J3 143.0 mm to (204.6, 47.4)
- moved J1 141.4 mm to (190.2, 57.0)
- moved R21 132.4 mm to (74.0, 60.9), turned to 270 degrees
- moved L3 131.4 mm to (97.0, 50.0)
- moved C2 130.3 mm to (94.0, 58.0), turned to 90 degrees
- moved C5 129.3 mm to (100.0, 58.0), turned to 90 degrees
- moved D2 125.7 mm to (97.0, 59.0)
- moved U2 125.7 mm to (97.0, 63.0)
- moved U1 119.9 mm to (87.0, 63.0)
- moved H3 117.5 mm to (97.0, 50.0)
- moved R20 116.2 mm to (130.5, 89.5)
- moved R23 115.1 mm to (135.5, 92.5)
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Connections:
- C4 pad 2: CONN_B -> CON_B
- C5 pad 2: CONN_C -> CON_C
- H1 pad 3: CONN_A -> CON_A
- H2 pad 3: CONN_B -> CON_B
- H3 pad 3: CONN_C -> CON_C
- J1 pad 1: CONN_B -> CON_B
- J2 pad 1: CONN_C -> CON_C
- J3 pad 1: CONN_A -> CON_A
- L1 pad 2: CONN_A -> CON_A
- L2 pad 2: CONN_B -> CON_B
- L3 pad 2: CONN_C -> CON_C
- U1 pad 6: CONN_B -> CON_B
- U2 pad 6: CONN_C -> CON_C
Other:
- board outline added: 38 x 54 mm
