File: XESC v1/XESC.sch (KiCad schematic (older format))
At the start: 96 parts, among them IC1 STM32G473CEU6, J1 PHASE A, J2 PHASE A, J3 PHASE A, J4 PWR_IN, J5 GND, J6 UART, J7 SWD, Q1 QM6015D, U1 IR2101, U2 IR2101, U3 IR2101, U4 ADP2302ARDZ-3.3, Y1 20MHz

Commit message: Add files via upload
Parts:
- removed C9: 4.7U, Capacitor_SMD:CP_Elec_4x3.9, symbol Device:C_Small
- removed H1, H2, H3, L1, L2, L3: IRFR3504ZPbF, Package_TO_SOT_SMD:TO-252-2, symbol Device:Q_NMOS_DGS
- removed R10, R11: 100, Resistor_SMD:R_0402_1005Metric, symbol Device:R_Small
- added C?: 4.7U, Capacitor_SMD:CP_Elec_4x3.9, symbol Device:C_Small
- added H3, L3: IRFR3504ZPbF, Package_TO_SOT_SMD:TO-252-2, symbol Device:Q_NMOS_GDS
- added Q? (x2): IRFI4212H, Package_TO_SOT_THT:TO-220F-5_P3.4x2.06mm_StaggerEven_Lead1.86mm_Vertical, symbol Transistor_FET:IRFI4212H
- added R? (x2): 100, Resistor_SMD:R_0402_1005Metric, symbol Device:R_Small
Connections:
- net CONN_A: now also Q?.3 (S1/D2)
- net CONN_B: now also Q?.3 (S1/D2)
- net CONN_C: now also H3.3 (S), L3.2 (D)
- net GND: now also C7.1, C?.1, L3.3 (S), Q?.1 (S2), Q?.1 (S2); no longer C7.2
- net H2: now also R?.2
- net L2: now also R?.2
- net VDD: now also C7.2, C?.2, H3.2 (D), Q?.5 (D1), Q?.5 (D1); no longer C7.1
- net at R6.1: now also Q?.4 (G1)
- net at R7.1: now also Q?.2 (G2)
- net at R8.1: now also H3.1 (G)
- net at R9.1: now also L3.1 (G)
- new net: Q?.4 (G1), R?.1
- new net: Q?.2 (G2), R?.1
Other:
- note added: "NVMFD6H840NL\nhttps://www.mouser.in/datasheet/2/308/NVMFD6H840NL-D-1634335.pdf"
- moved on the sheet: C7, R6, R7

Commit message: Add files via upload
Parts:
- removed C7, C8, C?: 4.7U, Capacitor_SMD:CP_Elec_4x3.9, symbol Device:C_Small
- removed Q? (x2): IRFI4212H, Package_TO_SOT_THT:TO-220F-5_P3.4x2.06mm_StaggerEven_Lead1.86mm_Vertical, symbol Transistor_FET:IRFI4212H
- removed R? (x2): 100, Resistor_SMD:R_0402_1005Metric, symbol Device:R_Small
- added H1, H2, L1, L2: IRFR3504ZPbF, Package_TO_SOT_SMD:TO-252-2, symbol Device:Q_NMOS_GDS
- added R10, R11: 100, Resistor_SMD:R_0805_2012Metric, symbol Device:R_Small
- C1, C2, C3, C4, C5, C6: footprint Capacitor_SMD:CP_Elec_4x3.9 -> Capacitor_SMD:C_0805_2012Metric_Pad1.15x1.40mm_HandSolder
- C10, C11, C12, C13, C14, C15, C16, C17, C18, C19, C20, C21, C22: footprint Capacitor_SMD:C_0201_0603Metric -> Capacitor_SMD:C_0805_2012Metric_Pad1.15x1.40mm_HandSolder
- C23, C24: footprint Capacitor_SMD:C_0201_0603Metric -> Capacitor_THT:CP_Radial_D25.0mm_P10.00mm_SnapIn
- D4, D5, D6, D7, D8: footprint LED_SMD:LED_0201_0603Metric -> LED_SMD:LED_0805_2012Metric_Pad1.15x1.40mm_HandSolder
- J1, J2, J3, J4, J5: footprint ASSETS:PAD_5X5 -> ASSETS:PAD_7X6.75
- R1, R12, R13, R14, R15, R16, R17, R18, R19, R2, R20, R21, R22, R23, R24, R25, R26, R27, R28, R3, R4, R5, R6, R7, R8, R9: footprint Resistor_SMD:R_0402_1005Metric -> Resistor_SMD:R_0805_2012Metric
Connections:
- net CONN_A: no longer J3.1 (Pin_1)
- net CONN_B: no longer C4.2, J1.1 (Pin_1), U1.6 (VS)
- net CONN_C: no longer C5.2, H3.3 (S), J2.1 (Pin_1), L3.2 (D), U2.6 (VS)
- net GND: now also L1.3 (S), L2.3 (S)
- net H2: now also R10.2
- net L2: now also R11.2
- net VDD: now also H1.2 (D), H2.2 (D)
- net at R6.1: now also H1.1 (G)
- net at R7.1: now also L1.1 (G)
- new net: H2.1 (G), R10.1
- new net: L2.1 (G), R11.1
- new net CON_A: H1.3 (S), J3.1 (Pin_1), L1.2 (D)
- new net CON_B: C4.2, H2.3 (S), J1.1 (Pin_1), L2.2 (D), U1.6 (VS)
- new net CON_C: C5.2, H3.3 (S), J2.1 (Pin_1), L3.2 (D), U2.6 (VS)
