File: Teseo GNSS Breakout/Teseo_Mod.kicad_pcb (KiCad board)
At the start: 2 copper layers, 32.8 x 13.5 mm, 16 parts, among them J1 SMA_Edge, J2 Conn_02x05_Counter_Clockwise, U1 TSLP_6_2, U2 B4327, U3 TESEO-LIV3F

Commit message: Add files via upload
Parts:
- U1: value TSLP_6_2 -> BGA725L6E6327FTSA1
- moved C5 110.2 mm to (55.8, 82.4)
- moved U3 109.9 mm to (49.4, 82.8)
- moved C3 109.9 mm to (56.4, 86.2)
- moved U2 109.9 mm to (58.2, 85.9)
- moved R1 109.6 mm to (56.2, 84.4), turned to 270 degrees
- moved C7 109.4 mm to (40.6, 86.0)
- moved L2 109.4 mm to (41.8, 85.6)
- moved C6 109.3 mm to (43.0, 86.1)
- moved J2 109.3 mm to (38.0, 88.0)
- moved C4 109.1 mm to (43.0, 83.4)
- moved J1 109.1 mm to (64.1, 82.8)
- moved C2 108.5 mm to (59.9, 87.2), turned to 90 degrees
- moved L1 107.5 mm to (59.9, 84.2)
- moved U1 107.4 mm to (60.4, 85.6), turned to 90 degrees
- moved C1 107.4 mm to (60.2, 82.8)
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Routing:
- net GND: track 31.4 -> 54.0 mm, vias 37 -> 31
- net VCC_RF: track 9.07 -> 2.79 mm, vias 2 -> 0
- net +3V3: track 3.86 -> 8.43 mm, vias 0 -> 1
- net SYS_RSTN: track 20.1 -> 24.7 mm
- net WAKE_UP: track 11.5 -> 14.6 mm, vias 0 -> 1
- net ANT_OFF: track 6.55 -> 8.71 mm
- net Net-(C1-Pad2): track 5.28 -> 3.56 mm
- net V_BAT: track 11.8 -> 10.3 mm, vias 2 -> 1
- net Net-(C6-Pad2): track 4.29 -> 5.14 mm
- net 1PPS: track 7.94 -> 7.31 mm
- net TX: track 7.80 -> 7.16 mm
- net RX: track 10.9 -> 10.3 mm
- net SCL: track 17.9 -> 17.4 mm, vias 2 -> 0
- net SDA: track 20.8 -> 21.1 mm, vias 2 -> 0
- added copper zone on Power_Plane, net +3V3
- added copper zone on Ground_Plane, net GND
Other:
- board size 32.8 x 13.5 mm -> 33 x 13.8 mm
- copper layers 2 -> 4
- net class Default: clearance 0.15 -> 0.12
- rule trace_clearance: 0.15 -> 0.12
