File: Teseo GNSS Breakout/Teseo_Mod.sch (KiCad schematic (older format))
At the start: 15 parts, among them J1 SMA_Edge, J2 Conn_02x05_Counter_Clockwise, U1 BGA725L6E6327FTSA1, U2 B4327, U3 TESEO-LIV3F

Commit message: Add files via upload
Changed lines of the file:
@@
 Text GLabel 9530 5280 0    50   Input ~ 0
 V_BAT
-Wire Wire Line
-	9750 5380 9560 5380
 $Comp
 L power:GND #PWR012
 U 1 1 5EC096D0
-P 9560 5380
-F 0 "#PWR012" H 9560 5130 50  0001 C CNN
-F 1 "GND" V 9565 5252 50  0000 R CNN
-F 2 "" H 9560 5380 50  0001 C CNN
-F 3 "" H 9560 5380 50  0001 C CNN
-	1    9560 5380
+P 9110 5380
+F 0 "#PWR012" H 9110 5130 50  0001 C CNN
+F 1 "GND" V 9115 5252 50  0000 R CNN
+F 2 "" H 9110 5380 50  0001 C CNN
+F 3 "" H 9110 5380 50  0001 C CNN
+	1    9110 5380
 	0    1    1    0
 $EndComp
-Wire Wire Line
-	9750 5480 9530 5480
 $Comp
 L power:+3.3V #PWR011
 U 1 1 5EC0B3F8
-P 9530 5480
-F 0 "#PWR011" H 9530 5330 50  0001 C CNN
-F 1 "+3.3V" V 9545 5608 50  0000 L CNN
-F 2 "" H 9530 5480 50  0001 C CNN
-F 3 "" H 9530 5480 50  0001 C CNN
-	1    9530 5480
+P 9080 5480
+F 0 "#PWR011" H 9080 5330 50  0001 C CNN
+F 1 "+3.3V" V 9095 5608 50  0000 L CNN
+F 2 "" H 9080 5480 50  0001 C CNN
+F 3 "" H 9080 5480 50  0001 C CNN
+	1    9080 5480
 	0    -1   -1   0
 $EndComp
@@
 Wire Wire Line
 	10250 5280 10450 5280
+Wire Wire Line
+	9110 5380 9170 5380
+Wire Wire Line
+	9080 5480 9110 5480
+$Comp
+L power:PWR_FLAG #FLG?
+U 1 1 5EBDA7F4
+P 8870 5620
+F 0 "#FLG?" H 8870 5695 50  0001 C CNN
+F 1 "PWR_FLAG" V 8870 5747 50  0000 L CNN
+F 2 "" H 8870 5620 50  0001 C CNN
+F 3 "~" H 8870 5620 50  0001 C CNN
+	1    8870 5620
+	0    -1   -1   0
+$EndComp
+$Comp
+L power:GNDPWR #PWR?
+U 1 1 5EBDAB47
+P 8950 5240
+F 0 "#PWR?" H 8950 5040 50  0001 C CNN
+F 1 "GNDPWR" V 8954 5131 50  0000 R CNN
+F 2 "" H 8950 5190 50  0001 C CNN
+F 3 "" H 8950 5190 50  0001 C CNN
+	1    8950 5240
+	0    1    1    0
+$EndComp
+Wire Wire Line
+	8950 5240 9170 5240
+Wire Wire Line
+	9170 5240 9170 5380
+Connection ~ 9170 5380
+Wire Wire Line
+	9170 5380 9750 5380
+Wire Wire Line
+	8870 5620 9110 5620
+Wire Wire Line
+	9110 5620 9110 5480
+Connection ~ 9110 5480
+Wire Wire Line
+	9110 5480 9750 5480
 $EndSCHEMATC
