File: Teseo GNSS Breakout/copy1.kicad_pcb (KiCad board)
At the start: 4 copper layers, 33 x 13.8 mm, 16 parts, among them J1 SMA_Edge, J2 Conn_02x05_Counter_Clockwise, U1 BGA725L6E6327FTSA1, U2 B4327, U3 TESEO-LIV3F

Commit message: Add files via upload
Parts:
- moved REF** 166.9 mm to (217.0, 128.0)
Routing:
- net GND: track 27.7 -> 12.0 mm, vias 14 -> 12
- net (no net): track 0.00 -> 11.7 mm
Other:
- board outline removed
Changed lines of the file:
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@@
   (general
     (thickness 1.6)
-    (drawings 23)
-    (tracks 108)
+    (drawings 19)
+    (tracks 104)
     (zones 0)
     (modules 16)
@@
   )
   (module Symbol:OSHW-Logo2_7.3x6mm_SilkScreen (layer B.Cu)
-    (at 56.2 83.2)
+    (at 217 128)
     (descr "Open Source Hardware Symbol")
     (tags "Logo Symbol OSHW")
@@
     )
   )
-  (gr_line (start 33.6 89.8) (end 33.6 76) (layer Edge.Cuts) (width 0.05))
-  (gr_line (start 66.6 89.8) (end 33.6 89.8) (layer Edge.Cuts) (width 0.05))
-  (gr_line (start 66.6 76) (end 66.6 89.8) (layer Edge.Cuts) (width 0.05))
-  (gr_line (start 33.6 76) (end 66.6 76) (layer Edge.Cuts) (width 0.05))
   (gr_line (start 66.6 76) (end 62.2 76) (layer Dwgs.User) (width 0.15))
   (gr_line (start 66.6 76.8) (end 66.6 76) (layer Dwgs.User) (width 0.15))
@@
   (gr_line (start 66.6 89.8) (end 66.6 77.8) (layer Dwgs.User) (width 0.15))
   (gr_line (start 33.6 89.8) (end 66.6 89.8) (layer Dwgs.User) (width 0.15))
-  (gr_text "6: RX\n7: TX\n8: SDA\n9: SCL\n10: RESET" (at 49 81.2 180) (layer B.SilkS)
+  (gr_text "6: RX\n7: TX\n8: SDA\n9: SCL\n10: RESET" (at 212.9 63.3 180) (layer B.SilkS)
     (effects (font (size 0.5 0.5) (thickness 0.125)) (justify mirror))
   )
-  (gr_text "1: VBAT\n2: GND\n3: 3.3V\n4: WAKEUP\n5: PPS\n" (at 49.2 85.6 180) (layer B.SilkS)
+  (gr_text "1: VBAT\n2: GND\n3: 3.3V\n4: WAKEUP\n5: PPS\n" (at 213.1 67.7 180) (layer B.SilkS)
     (effects (font (size 0.5 0.5) (thickness 0.125)) (justify mirror))
   )
-  (gr_text 9 (at 39.4 78.9) (layer F.SilkS)
+  (gr_text 9 (at 145 106.9) (layer F.SilkS)
     (effects (font (size 1 1) (thickness 0.15)))
   )
-  (gr_text 10 (at 36.7 79.2) (layer F.SilkS)
+  (gr_text 10 (at 142.3 107.2) (layer F.SilkS)
     (effects (font (size 1 0.75) (thickness 0.15)))
   )
-  (gr_text 7 (at 39.4 81.3) (layer F.SilkS)
+  (gr_text 7 (at 145 109.3) (layer F.SilkS)
     (effects (font (size 1 1) (thickness 0.15)))
   )
-  (gr_text 8 (at 36.7 81.4) (layer F.SilkS)
+  (gr_text 8 (at 142.3 109.4) (layer F.SilkS)
     (effects (font (size 1 1) (thickness 0.15)))
   )
-  (gr_text 5 (at 39.4 83.8) (layer F.SilkS)
+  (gr_text 5 (at 145 111.8) (layer F.SilkS)
     (effects (font (size 1 1) (thickness 0.15)))
   )
-  (gr_text 6 (at 36.7 83.9) (layer F.SilkS)
+  (gr_text 6 (at 142.3 111.9) (layer F.SilkS)
     (effects (font (size 1 1) (thickness 0.15)))
   )
-  (gr_text 3 (at 39.4 86.3) (layer F.SilkS)
+  (gr_text 3 (at 145 114.3) (layer F.SilkS)
     (effects (font (size 1 1) (thickness 0.15)))
   )
-  (gr_text 4 (at 36.8 86.4) (layer F.SilkS)
+  (gr_text 4 (at 142.4 114.4) (layer F.SilkS)
     (effects (font (size 1 1) (thickness 0.15)))
   )
-  (gr_text 2 (at 36.7 89) (layer F.SilkS)
+  (gr_text 2 (at 142.3 117) (layer F.SilkS)
     (effects (font (size 1 1) (thickness 0.15)))
   )
-  (gr_text 1 (at 39.8 89) (layer F.SilkS)
+  (gr_text 1 (at 145.4 117) (layer F.SilkS)
     (effects (font (size 1 1) (thickness 0.15)))
   )
-  (via micro (at 57 83) (size 0.8) (drill 0.4) (layers F.Cu Ground_Plane) (net 3))
-  (via micro (at 57 81) (size 0.8) (drill 0.4) (layers F.Cu Ground_Plane) (net 3))
-  (segment (start 57 79) (end 57 77) (width 1) (layer F.Cu) (net 3))
-  (segment (start 57 77) (end 59 77) (width 1) (layer F.Cu) (net 3))
-  (segment (start 61 77) (end 59 77) (width 1) (layer F.Cu) (net 3))
-  (segment (start 61 77) (end 63 77) (width 1) (layer F.Cu) (net 3))
-  (segment (start 63 77) (end 65 77) (width 1) (layer F.Cu) (net 3))
-  (segment (start 65 77) (end 65 78.679999) (width 1) (layer F.Cu) (net 3))
-  (segment (start 64.1 82.8) (end 60.54 82.8) (width 0.3) (layer F.Cu) (net 1))
-  (segment (start 59.9 83.88) (end 59.9 82.8) (width 0.3) (layer F.Cu) (net 2))
   (via micro (at 65 89) (size 0.8) (drill 0.4) (layers F.Cu Ground_Plane) (net 3))
   (via micro (at 63 89) (size 0.8) (drill 0.4) (layers F.Cu Ground_Plane) (net 3))
@@
   (via micro (at 63 77) (size 0.8) (drill 0.4) (layers F.Cu Ground_Plane) (net 3))
   (via micro (at 65 77) (size 0.8) (drill 0.4) (layers F.Cu Ground_Plane) (net 3))
-  (segment (start 57 81) (end 57 79) (width 1) (layer F.Cu) (net 3))
-  (segment (start 57 83) (end 57 81) (width 1) (layer F.Cu) (net 3))
+  (segment (start 57 79) (end 57 77) (width 1) (layer F.Cu) (net 0))
+  (segment (start 57 77) (end 59 77) (width 1) (layer F.Cu) (net 0))
+  (segment (start 61 77) (end 59 77) (width 1) (layer F.Cu) (net 0))
+  (segment (start 61 77) (end 63 77) (width 1) (layer F.Cu) (net 0))
+  (segment (start 63 77) (end 65 77) (width 1) (layer F.Cu) (net 0))
+  (segment (start 65 77) (end 65 78.679999) (width 1) (layer F.Cu) (net 0))
+  (segment (start 64.1 82.8) (end 60.54 82.8) (width 0.3) (layer F.Cu) (net 1))
+  (segment (start 59.9 83.88) (end 59.9 82.8) (width 0.3) (layer F.Cu) (net 2))
   (segment (start 59.9 86.65) (end 59.9 85.92501) (width 0.25) (layer F.Cu) (net 4))
   (segment (start 59.9 86.88) (end 59.9 86.65) (width 0.25) (layer F.Cu) (net 4))
@@
     (polygon
       (pts
-        (xy 65.5 79.2) (xy 64.5 79.2) (xy 64.472881 77.525) (xy 57.5 77.55) (xy 57.5 83.525)
-        (xy 56.5 83.475) (xy 56.5 76.5) (xy 65.5 76.5)
+        (xy 65.6 79.2) (xy 57.8 79.2) (xy 57.6 79.6) (xy 56.2 79.6) (xy 56.2 76.4)
+        (xy 65.6 76.4)
       )
     )
