File: LOGSX/MCU.sch (KiCad schematic (older format))
At the start: 1 part

Commit message: Add files via upload
Parts:
- removed J?: Conn_02x05_Counter_Clockwise, Connector_PinHeader_2.54mm:PinHeader_2x05_P2.54mm_Horizontal, symbol Connector_Generic:Conn_02x05_Counter_Clockwise
- added C1, C2, C3, C4, C5: 2.2pF, Capacitor_SMD:C_0201_0603Metric, symbol Device:C_Small
- added C10, C11, C12, C9: 2.2pF, Capacitor_SMD:C_0402_1005Metric, symbol Device:C_Small
- added C6: 1uF, Capacitor_SMD:C_0402_1005Metric, symbol Device:C_Small
- added C7, C8: 1pF, Capacitor_SMD:C_0201_0603Metric, symbol Device:C_Small
- added IC1: STM32G473CET6, Package_DFN_QFN:QFN-48-1EP_7x7mm_P0.5mm_EP5.45x5.45mm, symbol Regular_Use:STM32G473CET6
- added J1: Conn_01x02, Battery:BatteryHolder_Keystone_3008_1x2450, symbol Connector_Generic:Conn_01x02
- added JP1: SolderJumper_3_Open, Jumper:SolderJumper-3_P1.3mm_Open_Pad1.0x1.5mm_NumberLabels, symbol Jumper:SolderJumper_3_Open
- added R1: 1K7, Resistor_SMD:R_0402_1005Metric, symbol Device:R_Small
- added R2, R3: 4.7K, Resistor_SMD:R_0402_1005Metric, symbol Device:R_Small
- added TP1, TP2, TP3: TestPoint, TestPoint:TestPoint_Keystone_5015_Micro-Minature, symbol Connector:TestPoint
- added U1: W25Q32JVSS, Package_SO:SOIC-8_5.23x5.23mm_P1.27mm, symbol Memory_Flash:W25Q32JVSS
- added Y1: Crystal_GND24, Crystal:Crystal_SMD_Abracon_ABM8G-4Pin_3.2x2.5mm, symbol Device:Crystal_GND24
- added Y2: Crystal_GND24, Crystal:Crystal_SMD_SeikoEpson_MA506-4Pin_12.7x5.1mm, symbol Device:Crystal_GND24
Connections:
- net +3V3: now also C10.1, C11.1, C12.1, C5.2, C6.1, C9.1, IC1.20 (VREF+), IC1.21 (VDDA), IC1.24 (VDD_1), IC1.36 (VDD_2), IC1.48 (VDD_3), R1.1, R2.1, R3.1, U1.8 (VCC)
- net 1PPS: now also IC1.18 (PB2)
- net GND: now also C1.2, C10.2, C11.2, C12.2, C2.2, C3.2, C4.1, C5.1, C6.2, C7.2, C8.2, C9.2, IC1.19 (VSSA), IC1.23 (VSS_1), IC1.35 (VSS_2), IC1.47 (VSS_3), J1.1 (Pin_1), JP1.3 (B), TP3.1, U1.4 (GND), Y1.2, Y1.4, Y2.2, Y2.4
- net RX: now also IC1.40 (PB3)
- net SCL: now also IC1.31 (PA9), R2.2
- net SDA: now also IC1.30 (PA8), R3.2
- net SYS_RSTN: now also IC1.29 (PB15)
- net TX: now also IC1.41 (PB4)
- net V_BAT: now also C4.2, IC1.1 (VBAT), J1.2 (Pin_2)
- net WAKE_UP: now also IC1.17 (PB1)
- new net: C3.1, IC1.7 (PG10-NRST), JP1.2 (C)
- new net: JP1.1 (A), R1.2
- new net ALM: IC1.28 (PB14)
- new net FLASH_NSS: IC1.25 (PB11), U1.1 (~CS)
- new net LoRa_NSS: IC1.12 (PA4)
- new net LoRa_RESET: IC1.16 (PB0)
- new net MISO: IC1.14 (PA6), U1.2 (DO(IO1))
- new net MOSI: IC1.15 (PA7), U1.5 (DI(IO0))
- new net OSC32_IN: C7.1, IC1.3 (PC14-OSC32_IN), Y2.1
- new net OSC32_OUT: C8.1, IC1.4 (PC15-_OSC32_OUT), Y2.3
- new net OSC_IN: C1.1, IC1.5 (PF0-OSC_IN), Y1.1
- new net OSC_OUT: C2.1, IC1.6 (PF1-OSC_OUT), Y1.3
- new net SCK: IC1.13 (PA5), U1.6 (CLK)
- new net SWCLK: IC1.38 (PA14), TP1.1
- new net SWDIO: IC1.37 (PA13), TP2.1
- no-connect marks 0 -> 19

Commit message: Add files via upload
Parts:
- removed IC1: STM32G473CET6, Package_DFN_QFN:QFN-48-1EP_7x7mm_P0.5mm_EP5.45x5.45mm, symbol Regular_Use:STM32G473CET6
- removed J1: Conn_01x02, Battery:BatteryHolder_Keystone_3008_1x2450, symbol Connector_Generic:Conn_01x02
- removed Y1: Crystal_GND24, Crystal:Crystal_SMD_Abracon_ABM8G-4Pin_3.2x2.5mm, symbol Device:Crystal_GND24
- removed Y2: Crystal_GND24, Crystal:Crystal_SMD_SeikoEpson_MA506-4Pin_12.7x5.1mm, symbol Device:Crystal_GND24
- added U9: STM32F103C8Tx, Package_QFP:LQFP-48-1EP_7x7mm_P0.5mm_EP3.6x3.6mm, symbol MCU_ST_STM32F1:STM32F103C8Tx
- added Y1, Y2: Crystal_GND23, Crystal:Crystal_SMD_Abracon_ABM8G-4Pin_3.2x2.5mm, symbol Device:Crystal_GND23
Connections:
- net V_BAT is gone; now on net +3V3: C4.2
- net +3V3: now also U9.1 (VBAT), U9.24 (VDD), U9.36 (VDD), U9.44 (BOOT0), U9.48 (VDD), U9.9 (VDDA)
- net 1PPS: now also U9.32 (PA11)
- net ALM: now also U9.45 (PB8)
- net FLASH_NSS: now also U9.29 (PA8)
- net GND: now also U9.23 (VSS), U9.35 (VSS), U9.47 (VSS), U9.8 (VSSA), Y1.2, Y1.3, Y2.2, Y2.3
- net LoRa_NSS: now also U9.14 (PA4)
- net LoRa_RESET: now also U9.27 (PB14)
- net MISO: now also U9.16 (PA6)
- net MOSI: now also U9.17 (PA7)
- net OSC32_IN: now also U9.3 (PC14), Y2.1
- net OSC32_OUT: now also U9.4 (PC15), Y2.4
- net OSC_IN: now also U9.5 (PD0), Y1.1
- net OSC_OUT: now also U9.6 (PD1), Y1.4
- net RX: now also U9.30 (PA9)
- net SCK: now also U9.15 (PA5)
- net SCL: now also U9.42 (PB6)
- net SDA: now also U9.43 (PB7)
- net SWCLK: now also U9.37 (PA14)
- net SWDIO: now also U9.34 (PA13)
- net SYS_RSTN: now also U9.28 (PB15)
- net TX: now also U9.31 (PA10)
- net WAKE_UP: now also U9.33 (PA12)
- net at C3.1, JP1.2 (C): now also U9.7 (NRST)
Other:
- moved on the sheet: C3, C4, JP1, R1, R2, R3
