File: LOGSX/Radio.sch (KiCad schematic (older format))
At the start: 45 parts

Commit message: Add files via upload
Parts:
- removed R?: 1K, symbol Device:R_Small
- added C46, C47: 2.2pF, Capacitor_SMD:C_0201_0603Metric, symbol Device:C_Small
- added Y3: Crystal_GND24, Crystal:Crystal_SMD_Abracon_ABM8G-4Pin_3.2x2.5mm, symbol Device:Crystal_GND24
- R10: renamed from R?; footprint Inductor_SMD:L_0201_0603Metric -> Resistor_SMD:R_0402_1005Metric
- R11, R9: renamed from R?; footprint (none) -> Resistor_SMD:R_0402_1005Metric
- U7: renamed from U?; footprint (none) -> ASSETS:PE4259_sc70
- gave numbers to parts that had none: 40
Connections:
- net GND: now also C46.2, C47.2, Y3.2, Y3.4
- net PA_BOOST: now also U6.27 (PA_BOOST)
- net VR_PA: now also U6.28 (VR_PA)
- net XTA: now also C47.1, Y3.1
- net XTB: now also C46.1, Y3.3
- net RF_MOD: no longer names the net of U6.21 (RF_MOD/NC)
- no-connect marks 7 -> 8

Commit message: Add files via upload
Parts:
- removed Y3: Crystal_GND24, Crystal:Crystal_SMD_Abracon_ABM8G-4Pin_3.2x2.5mm, symbol Device:Crystal_GND24
- added Y3: Crystal_GND23, Crystal:Crystal_SMD_Abracon_ABM8G-4Pin_3.2x2.5mm, symbol Device:Crystal_GND23
Connections:
- net V_BAT is gone; now on net +3V3: C28.2, U4.6 (VBATT)
- net GND: now also J4.2_1 (GND), J4.2_2 (GND), J4.3_1 (GND), J4.3_2 (GND), Y3.2, Y3.3
- net XTA: now also Y3.1
- net XTB: now also Y3.4
Changed lines of the file:
@@
 	-1   0    0    1
 $EndComp
-Text GLabel 4240 860  0    50   Input ~ 0
-V_BAT
 Wire Wire Line
 	4440 860  4240 860
@@
 NoConn ~ 3460 7590
 $Comp
-L Device:Crystal_GND24 Y?
-U 1 1 5ECD13DD
-P 6670 6520
-AR Path="/5EBFF6BB/5ECD13DD" Ref="Y?"  Part="1"
-AR Path="/5EC12809/5ECD13DD" Ref="Y3"  Part="1"
-F 0 "Y3" V 6680 5910 50  0000 L CNN
-F 1 "Crystal_GND24" V 6760 5470 50  0000 L CNN
-F 2 "Crystal:Crystal_SMD_Abracon_ABM8G-4Pin_3.2x2.5mm" H 6670 6520 50  0001 C CNN
-F 3 "~" H 6670 6520 50  0001 C CNN
-	1    6670 6520
-	0    -1   1    0
-$EndComp
-$Comp
 L power:GND #PWR?
 U 1 1 5ECD13E3
@@
 Text GLabel 5870 6880 0    50   Input ~ 0
 XTB
+$Comp
+L power:GND #PWR0101
+U 1 1 5EBEFB0A
+P 1370 9260
+F 0 "#PWR0101" H 1370 9010 50  0001 C CNN
+F 1 "GND" H 1375 9087 50  0000 C CNN
+F 2 "" H 1370 9260 50  0001 C CNN
+F 3 "" H 1370 9260 50  0001 C CNN
+	1    1370 9260
+	1    0    0    -1
+$EndComp
+$Comp
+L Device:Crystal_GND23 Y?
+U 1 1 5EC534F0
+P 6670 6520
+AR Path="/5EBFF6BB/5EC534F0" Ref="Y?"  Part="1"
+AR Path="/5EC12809/5EC534F0" Ref="Y3"  Part="1"
+F 0 "Y3" V 6624 6764 50  0000 L CNN
+F 1 "Crystal_GND23" V 6715 6764 50  0000 L CNN
+F 2 "Crystal:Crystal_SMD_Abracon_ABM8G-4Pin_3.2x2.5mm" H 6670 6520 50  0001 C CNN
+F 3 "~" H 6670 6520 50  0001 C CNN
+	1    6670 6520
+	0    1    1    0
+$EndComp
+$Comp
+L power:+3.3V #PWR0103
+U 1 1 5EC638D1
+P 4240 860
+F 0 "#PWR0103" H 4240 710 50  0001 C CNN
+F 1 "+3.3V" V 4255 988 50  0000 L CNN
+F 2 "" H 4240 860 50  0001 C CNN
+F 3 "" H 4240 860 50  0001 C CNN
+	1    4240 860
+	0    -1   -1   0
+$EndComp
 $EndSCHEMATC
